File: ver3/dippy.kicad_pcb (KiCad board)
At the start: 2 copper layers, 29.5 x 68.7 mm, 22 parts, among them J1 Conn_01x02_Female, J2 Screw_Terminal_01x03, J3 Screw_Terminal_01x04, J4 Conn_Coaxial, J5 Conn_02x03_Odd_Even, U1 ATmega328P-PU-C, U2 RFM95W-915S2, U3 MCP1700-3302E_SOT23, Y1 Crystal

Commit message: update
Parts:
- added H3: MountingHole, MountingHole:MountingHole_2.7mm_M2.5, F.Cu at (142.9, 112.0)
- added H4: MountingHole, MountingHole:MountingHole_2.7mm_M2.5, F.Cu at (119.5, 66.5)
- moved J5 4.43 mm to (141.0, 121.1)
- moved J1 2.93 mm to (118.7, 71.9)
- moved FTDI1 1.88 mm to (124.8, 67.7)
- moved H2 1.83 mm to (119.5, 112.0)
- moved C3 0.38 mm to (135.6, 97.2)
- moved H1 0.09 mm to (143.0, 66.5)
Routing:
- net GND: track 199.2 -> 190.3 mm
- net MISO: track 45.0 -> 51.3 mm
- net Net-(C1-Pad1): track 56.9 -> 61.0 mm
- net SCK: track 50.8 -> 54.3 mm
- net TX0: track 20.1 -> 23.3 mm
- net Net-(J4-Pad1): track 18.7 -> 16.1 mm
- net MOSI: track 47.1 -> 44.6 mm
- net RX0: track 16.4 -> 18.7 mm, vias 0 -> 1
- net Net-(C1-Pad2): track 7.18 -> 6.58 mm
- net VIN: track 41.5 -> 41.0 mm, vias 1 -> 2
- net VCC: track 114.7 -> 114.6 mm, vias 2 -> 1
Other:
- board text added: "3V"
- board text added: "A0"
- board text added: "A1"
- board text added: "A2"
- board text added: "G"
- board text added: "RX"
- board text added: "TX"
- board text added: "VCC"
- board text added: "VIN"

Commit message: update
Routing:
- net (no net): track 0.00 -> 4.66 mm, vias 0 -> 2
- net GND: track 190.3 -> 189.6 mm
Other:
- board text added: "A3"
- board text added: "A4"
- board text added: "ANT"
- board text added: "DR"

Commit message: update
Parts:
- added J6: Screw_Terminal_01x04, TerminalBlock_Phoenix:TerminalBlock_Phoenix_PT-1,5-4-3.5-H_1x04_P3.50mm_Horizontal, F.Cu at (140.9, 91.0)
- added J7: Conn_01x02_Female, Connector_PinSocket_2.54mm:PinSocket_1x02_P2.54mm_Vertical, B.Cu at (130.9, 86.9)
- moved J3 31.8 mm to (119.2, 80.1), turned to 270 degrees
- moved R3 23.3 mm to (116.1, 101.5), turned to 270 degrees
- moved J2 19.0 mm to (140.8, 106.5)
- moved R2 18.4 mm to (144.9, 94.5), turned to 180 degrees
- moved C4 10.5 mm to (124.0, 76.5), turned to 180 degrees
- moved C2 8.04 mm to (121.3, 71.5)
- moved C5 4.55 mm to (119.1, 94.6), turned to 270 degrees
- moved J1 3.63 mm to (116.1, 74.4), turned to 180 degrees
- moved C1 3.30 mm to (142.2, 74.0)
- moved Y1 3.24 mm to (121.0, 101.4)
- moved R1 3.17 mm to (134.8, 74.5)
- moved R5 3.08 mm to (139.8, 71.9)
- moved H4 2.47 mm to (117.2, 65.5)
- moved U3 2.46 mm to (129.2, 72.5)
- moved H2 2.34 mm to (117.2, 112.5)
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Connections:
- J2 pad 2: A2 -> VCC
- J2 pad 3: VCC -> A0
- J3 pad 3: A0 -> D3
- J3 pad 4: A1 -> D4
- R2 pad 2: A2 -> A0
- R3 pad 2: A0 -> D4
- R4 pad 2: A5 -> A3
- R5 pad 1: A5 -> A3
- U1 pad 26: (no net) -> A3
- U1 pad 27: (no net) -> A4
- U1 pad 4: (no net) -> D2
- U1 pad 6: (no net) -> D4
- U2 pad 14: D3 -> D2
Routing:
- net D2: track 0.00 -> 41.5 mm, vias 0 -> 3
- net D3: track 38.5 -> 7.56 mm, vias 3 -> 0
- net VCC: track 114.6 -> 144.6 mm, vias 1 -> 2
- net A3: track 0.00 -> 27.5 mm, vias 0 -> 2
- net D4: track 0.00 -> 27.4 mm
- net A2: track 23.9 -> 2.51 mm
- net A5: track 20.8 -> 7.98 mm
- net A0: track 24.1 -> 13.9 mm
- net A4: track 0.00 -> 9.37 mm
- net GND: track 189.6 -> 198.3 mm, vias 10 -> 8
- net VIN: track 41.0 -> 33.5 mm, vias 2 -> 0
- net MISO: track 51.3 -> 44.4 mm
- net A1: track 9.38 -> 2.51 mm
- net Net-(C1-Pad1): track 61.0 -> 65.8 mm
- net Net-(U1-Pad10): track 4.83 -> 7.03 mm
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Other:
- board size 29.5 x 68.7 mm -> 31.7 x 69.7 mm
- board text added: "1"
- board text added: "9"
- board text added: "D3"
- board text added: "D4"
- board text added: "D5"
- board text added: "DTR"
- board text added: "GND"
- board text added: "MI"
- board text added: "MO"
- board text added: "RFM9x"
- board text added: "RST"
- board text added: "SCK"
- board text added: "SCL"
- board text added: "SDA"
- board text removed: "A3"
- board text removed: "A4"
- board text removed: "DR"
- board text removed: "VCC"

Commit message: update
Parts:
- added D1: LED, LED_THT:LED_D3.0mm, F.Cu at (116.5, 105.7)
- added G***: LOGO, footprints:moth4, F.Cu at (137.0, 111.2)
- added R6: 300R, Resistor_THT:R_Axial_DIN0204_L3.6mm_D1.6mm_P5.08mm_Horizontal, F.Cu at (115.3, 102.1)
- moved C5 2.10 mm to (121.2, 94.4)
- moved R3 1.49 mm to (117.5, 100.9), turned to 90 degrees
- moved Y1 1.30 mm to (121.6, 102.5)
Connections:
- U1 pad 11: (no net) -> D5
Routing:
- net D5: track 0.00 -> 14.5 mm, vias 0 -> 1
- net D4: track 27.4 -> 13.0 mm
- net GND: track 198.3 -> 211.0 mm
- net Net-(D1-Pad1): track 0.00 -> 4.11 mm
- net VCC: track 144.6 -> 140.6 mm
- net A3: track 27.5 -> 24.3 mm
- net (no net): track 2.78 -> 0.00 mm, vias 1 -> 0
- net A5: track 7.98 -> 10.7 mm
- net Net-(C1-Pad1): track 65.8 -> 67.7 mm
- net Net-(U1-Pad9): track 5.48 -> 6.40 mm
- net Net-(U1-Pad10): track 7.03 -> 7.92 mm
- net A4: track 9.37 -> 10.2 mm
Other:
- board text added: "..::DIY Radio Node::.."
- board text added: "AT"
- board text added: "mothbot"
- board text added: "pvos.org/"
- board text added: "ver 0.1"
- board text removed: "ANT"
- board text removed: "GND"
