File: ver3/dippy.kicad_pcb (KiCad board)
At the start: 2 copper layers, 33.7 x 73.7 mm, 37 parts, among them J1 Screw_Terminal_01x02, J10 Conn_01x04_Female, J11 Conn_01x03_Female, J2 Screw_Terminal_01x03, J3 Screw_Terminal_01x04, J4 Conn_Coaxial, J5 Conn_02x03_Odd_Even, J6 Conn_01x04_Female, J7 Conn_01x03_Female, J8 Screw_Terminal_01x04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

Commit message: update
Parts:
- removed H3, H4: MountingHole, MountingHole:MountingHole_2.7mm_M2.5
- C1, C2, C3, C4, C6: footprint Capacitor_THT:C_Disc_D3.0mm_W1.6mm_P2.50mm -> Capacitor_THT:C_Disc_D4.3mm_W1.9mm_P5.00mm
- D1: footprint LED_THT:LED_D3.0mm -> LED_THT:LED_D5.0mm
- J1: footprint TerminalBlock_Phoenix:TerminalBlock_Phoenix_PT-1,5-2-3.5-H_1x02_P3.50mm_Horizontal -> TerminalBlock_Phoenix:TerminalBlock_Phoenix_PT-1,5-2-5.0-H_1x02_P5.00mm_Horizontal
- J11, J7: footprint Connector_PinHeader_2.54mm:PinHeader_1x03_P2.54mm_Vertical -> Connector_PinSocket_2.54mm:PinSocket_1x03_P2.54mm_Vertical
- J2: footprint TerminalBlock_Phoenix:TerminalBlock_Phoenix_PT-1,5-3-3.5-H_1x03_P3.50mm_Horizontal -> TerminalBlock_Phoenix:TerminalBlock_Phoenix_PT-1,5-3-5.0-H_1x03_P5.00mm_Horizontal
- J3, J8: footprint TerminalBlock_Phoenix:TerminalBlock_Phoenix_PT-1,5-4-3.5-H_1x04_P3.50mm_Horizontal -> TerminalBlock_Phoenix:TerminalBlock_Phoenix_PT-1,5-4-5.0-H_1x04_P5.00mm_Horizontal
- R1, R2, R3, R4, R5, R6, R7, R8: footprint Resistor_THT:R_Axial_DIN0204_L3.6mm_D1.6mm_P5.08mm_Horizontal -> Resistor_THT:R_Axial_DIN0204_L3.6mm_D1.6mm_P7.62mm_Horizontal
- moved H1 281.6 mm to (-129.0, -3.65)
- moved J4 258.3 mm to (-108.0, 70.3)
- moved U2 255.4 mm to (-130.1, 56.3)
- moved AT1 253.6 mm to (-108.0, 65.6)
- moved J1 253.6 mm to (-125.0, 3.52)
- moved J9 251.5 mm to (-111.0, 3.80), turned to 90 degrees
- moved R2 251.0 mm to (-96.7, 35.5), turned to 0 degrees
- moved C1 250.9 mm to (-107.2, 15.8), turned to 0 degrees
- moved C4 250.5 mm to (-122.7, 13.9), turned to 180 degrees
- moved U3 250.4 mm to (-118.3, 15.3)
- moved D1 248.7 mm to (-125.7, 49.4)
- moved FTDI1 248.0 mm to (-114.8, -2.70)
- moved R8 247.7 mm to (-108.5, 12.4)
- moved J3 247.7 mm to (-125.0, 22.1)
- moved R4 247.7 mm to (-97.7, 7.50)
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Connections:
- SW1 pad 2: GND -> RST
- SW1 pad 3: RST -> GND
Routing:
- net GND: track 233.2 -> 0.00 mm, vias 8 -> 0
- net VCC: track 168.3 -> 0.00 mm, vias 3 -> 0
- net RST: track 72.8 -> 0.00 mm, vias 1 -> 0
- net SCK: track 53.6 -> 0.00 mm, vias 3 -> 0
- net VIN: track 47.1 -> 0.00 mm
- net MOSI: track 44.6 -> 0.00 mm, vias 1 -> 0
- net MISO: track 44.4 -> 0.00 mm, vias 2 -> 0
- net D2: track 41.5 -> 0.00 mm, vias 3 -> 0
- net TX0: track 36.7 -> 0.00 mm, vias 2 -> 0
- net RX0: track 32.4 -> 0.00 mm, vias 2 -> 0
- net A3: track 29.8 -> 0.00 mm, vias 1 -> 0
- net D7: track 22.4 -> 0.00 mm
- net D8: track 19.4 -> 0.00 mm, vias 2 -> 0
- net A4: track 17.4 -> 0.00 mm
- net Net-(C1-Pad2): track 17.0 -> 0.00 mm, vias 1 -> 0
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Other:
- board size 33.7 x 73.7 mm -> 46.6 x 79.2 mm
- board text removed: "..::DIY Radio Node::.."
- board text removed: "1/GND"
- board text removed: "2/MISO"
- board text removed: "3V"
- board text removed: "9/ANT"
- board text removed: "A0"
- board text removed: "A1"
- board text removed: "A2"
- board text removed: "A4"
- board text removed: "A5"
- board text removed: "ANT"
- board text removed: "D3"
- board text removed: "D4"
- board text removed: "DC-DC"
- board text removed: "DTR"
- board text removed: "FTDI"
- board text removed: "G"
- board text removed: "GND"
- board text removed: "MI"
- board text removed: "MO"
- board text removed: "RFM9x"
- board text removed: "RST"
- board text removed: "RX"
- board text removed: "SCK"
- board text removed: "TX"
- board text removed: "VCC"
- board text removed: "VIN"
- board text removed: "mothbot"
- board text removed: "pvos.org/"
- board text removed: "ver 2"

Commit message: update
Parts:
- moved AT1 5.62 mm to (-110.8, 70.5)
- moved J4 3.48 mm to (-104.6, 70.1)
Changed lines of the file:
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@@
   )
   (module Connector_Coaxial:SMA_Samtec_SMA-J-P-X-ST-EM1_EdgeMount (layer F.Cu)
-    (at -108.05 70.325)
+    (at -104.575 70.125)
     (descr "Connector SMA, 0Hz to 20GHz, 50Ohm, Edge Mount (http://suddendocs.samtec.com/prints/sma-j-p-x-st-em1-mkt.pdf)")
     (tags "SMA Straight Samtec Edge Mount")
@@
   )
   (module Connector_PinSocket_2.54mm:PinSocket_1x01_P2.54mm_Vertical (layer F.Cu)
-    (at -108 65.6)
+    (at -110.75 70.5)
     (descr "Through hole straight socket strip, 1x01, 2.54mm pitch, single row (from Kicad 4.0.7), script generated")
     (tags "Through hole socket strip THT 1x01 2.54mm single row")

Commit message: update
Parts:
- added H3: MountingHole, MountingHole:MountingHole_2.7mm_M2.5, F.Cu at (-89.1, -3.50)
- added H4: MountingHole, MountingHole:MountingHole_2.7mm_M2.5, F.Cu at (-129.2, 69.3)
- moved C1 22.0 mm to (-94.2, -2.03), turned to 180 degrees
- moved R4 20.0 mm to (-117.3, 10.7), turned to 90 degrees
- moved R5 17.0 mm to (-114.8, 3.05), turned to 270 degrees
- moved D1 9.57 mm to (-128.8, 58.4)
- moved AT1 8.14 mm to (-102.6, 70.4)
- moved J4 8.06 mm to (-96.5, 70.1)
- moved U2 7.97 mm to (-122.2, 57.1)
- moved Y1 6.45 mm to (-117.3, 44.7), turned to 270 degrees
- moved J11 5.18 mm to (-99.8, 50.8), turned to 180 degrees
- moved C6 5.11 mm to (-99.6, 34.0), turned to 270 degrees
- moved C3 5.04 mm to (-102.4, 39.1), turned to 90 degrees
- moved U3 4.54 mm to (-113.8, 16.0), turned to 180 degrees
- moved SW1 4.43 mm to (-94.0, 7.87)
- moved R1 4.09 mm to (-97.0, 8.13)
- moved C2 3.63 mm to (-124.2, 13.7)
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Routing:
- net GND: track 0.00 -> 298.2 mm, vias 0 -> 4
- net VCC: track 0.00 -> 168.1 mm, vias 0 -> 1
- net RST: track 0.00 -> 107.7 mm, vias 0 -> 1
- net A3: track 0.00 -> 107.0 mm, vias 0 -> 1
- net MOSI: track 0.00 -> 54.6 mm, vias 0 -> 5
- net MISO: track 0.00 -> 54.3 mm, vias 0 -> 3
- net SCK: track 0.00 -> 47.1 mm, vias 0 -> 3
- net VIN: track 0.00 -> 41.4 mm
- net D2: track 0.00 -> 38.1 mm
- net A4: track 0.00 -> 36.5 mm
- net D5: track 0.00 -> 35.3 mm, vias 0 -> 1
- net TX0: track 0.00 -> 34.7 mm
- net A0: track 0.00 -> 33.0 mm
- net RX0: track 0.00 -> 29.7 mm
- net D7: track 0.00 -> 29.7 mm, vias 0 -> 2
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Other:
- outline, holes or cut-outs redrawn

Commit message: update
Parts:
- moved R2 1.80 mm to (-96.8, 38.4)
- moved J11 1.73 mm to (-99.8, 52.5)
- moved J2 1.73 mm to (-93.4, 54.6)
- moved C6 0.09 mm to (-99.6, 34.1)
Routing:
- net GND: track 298.2 -> 301.6 mm
- net RST: track 107.7 -> 109.5 mm, vias 1 -> 3
- net A0: track 33.0 -> 34.5 mm
- net VCC: track 168.1 -> 169.4 mm

Commit message: update
Parts:
- moved H1 0.66 mm to (-129.4, -3.88)
- moved H3 0.55 mm to (-88.7, -3.88)
- moved H4 0.21 mm to (-129.4, 69.5)
- moved H2 0.20 mm to (-88.7, 69.5)
Routing:
- net GND: track 301.6 -> 315.2 mm
Other:
- outline, holes or cut-outs redrawn
Changed lines of the file:
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@@
   (general
     (thickness 1.6)
-    (drawings 19)
-    (tracks 390)
+    (drawings 22)
+    (tracks 393)
     (zones 0)
     (modules 37)
@@
   )
   (module MountingHole:MountingHole_2.7mm_M2.5 (layer F.Cu)
-    (at -129.25 69.35)
+    (at -129.4 69.5)
     (descr "Mounting Hole 2.7mm, no annular, M2.5")
     (tags "mounting hole 2.7mm no annular m2.5")
@@
   )
   (module MountingHole:MountingHole_2.7mm_M2.5 (layer F.Cu)
-    (at -89.075 -3.5)
+    (at -88.675 -3.875)
     (descr "Mounting Hole 2.7mm, no annular, M2.5")
     (tags "mounting hole 2.7mm no annular m2.5")
@@
   )
   (module MountingHole:MountingHole_2.7mm_M2.5 (layer F.Cu)
-    (at -88.775 69.35)
+    (at -88.65 69.5)
     (descr "Mounting Hole 2.7mm, no annular, M2.5")
     (tags "mounting hole 2.7mm no annular m2.5")
@@
   )
   (module MountingHole:MountingHole_2.7mm_M2.5 (layer F.Cu)
-    (at -128.8 -3.6)
+    (at -129.4 -3.875)
     (descr "Mounting Hole 2.7mm, no annular, M2.5")
     (tags "mounting hole 2.7mm no annular m2.5")
@@
     )
   )
+  (gr_arc (start -129.227223 -3.725001) (end -129.977222 -6.8) (angle -64.45097618) (layer Edge.Cuts) (width 0.05))
+  (gr_arc (start -88.799999 -3.700001) (end -85.725 -4.45) (angle -64.45097618) (layer Edge.Cuts) (width 0.05))
+  (gr_arc (start -88.822777 69.325001) (end -88.072778 72.4) (angle -64.45097618) (layer Edge.Cuts) (width 0.05))
+  (gr_arc (start -129.25 69.3) (end -132.324999 70.049999) (angle -64.45097618) (layer Edge.Cuts) (width 0.05))
   (gr_line (start -99.825 26.975) (end -99.825 47.425) (layer Dwgs.User) (width 0.15))
   (gr_line (start -99.822 41.91) (end -99.822 9.398) (layer F.SilkS) (width 0.05))
@@
     (arrow2b (pts (xy -99.822 -19.304) (xy -100.948504 -18.717579)))
   )
-  (gr_line (start -132.325 -6.8) (end -85.725 -6.8) (layer Edge.Cuts) (width 0.05))
-  (gr_line (start -85.725 72.4) (end -132.325 72.4) (layer Edge.Cuts) (width 0.05))
-  (gr_line (start -85.725 -6.8) (end -85.725 72.4) (layer Edge.Cuts) (width 0.05))
-  (gr_line (start -132.325 -6.8) (end -132.325 -5.875) (layer Edge.Cuts) (width 0.05))
-  (gr_line (start -132.325 -5.875) (end -132.325 72.4) (layer Edge.Cuts) (width 0.05))
+  (gr_line (start -129.975 -6.8) (end -88.15 -6.8) (layer Edge.Cuts) (width 0.05))
+  (gr_line (start -88.075 72.4) (end -129.9 72.4) (layer Edge.Cuts) (width 0.05))
+  (gr_line (start -85.725 -4.45) (end -85.725 69.975) (layer Edge.Cuts) (width 0.05))
+  (gr_line (start -132.325 -4.374535) (end -132.325 70.05) (layer Edge.Cuts) (width 0.05))
   (gr_line (start -103.589 3.578) (end -100.289 3.578) (layer F.SilkS) (width 0.15))
   (gr_line (start -111.939 11.128) (end -100.289 11.128) (layer F.SilkS) (width 0.15))
@@
   (segment (start -88.646 65.278) (end -88.646 60.706) (width 1) (layer B.Cu) (net 4))
   (via (at -88.646 60.706) (size 0.8) (drill 0.4) (layers F.Cu B.Cu) (net 4))
-  (segment (start -119.634 57.69) (end -119.634 69.596) (width 1) (layer F.Cu) (net 4))
   (segment (start -95.465 52.525) (end -93.375 54.615) (width 1) (layer F.Cu) (net 4))
   (segment (start -99.797 52.525) (end -95.465 52.525) (width 1) (layer F.Cu) (net 4))
@@
   (segment (start -91.3555 40.3945) (end -90.6695 40.3945) (width 1) (layer B.Cu) (net 4))
   (segment (start -95.025 36.725) (end -91.3555 40.3945) (width 1) (layer B.Cu) (net 4))
+  (segment (start -106.174 69.15) (end -119.243 69.15) (width 1) (layer F.Cu) (net 4))
+  (segment (start -119.634 57.69) (end -119.634 68.759) (width 1) (layer F.Cu) (net 4))
+  (segment (start -119.243 69.15) (end -119.634 68.759) (width 1) (layer F.Cu) (net 4))
+  (segment (start -119.634 68.759) (end -119.634 69.596) (width 1) (layer F.Cu) (net 4))
   (segment (start -109.695 4.572) (end -108.689 5.578) (width 1) (layer F.Cu) (net 5))
   (segment (start -109.695 -2.7) (end -109.695 4.572) (width 1) (layer F.Cu) (net 5))

Commit message: update
Parts:
- moved C6 0.88 mm to (-99.5, 35.0)
- moved C3 0.88 mm to (-102.3, 40.0)
- moved R2 0.63 mm to (-96.8, 37.7)
Routing:
- net VCC: track 169.4 -> 170.9 mm
- net Net-(C3-Pad1): track 3.37 -> 4.73 mm
- net A3: track 107.0 -> 106.0 mm
Changed lines of the file:
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@@
     (thickness 1.6)
     (drawings 22)
-    (tracks 393)
+    (tracks 391)
     (zones 0)
     (modules 37)
@@
   )
   (module Capacitor_THT:C_Disc_D4.3mm_W1.9mm_P5.00mm (layer F.Cu)
-    (at -102.362 39.116 90)
+    (at -102.287 39.991 90)
     (descr "C, Disc series, Radial, pin pitch=5.00mm, , diameter*width=4.3*1.9mm^2, Capacitor, http://www.vishay.com/docs/45233/krseries.pdf")
     (tags "C Disc series Radial pin pitch 5.00mm  diameter 4.3mm width 1.9mm Capacitor")
@@
   )
   (module Resistor_THT:R_Axial_DIN0204_L3.6mm_D1.6mm_P7.62mm_Horizontal (layer F.Cu)
-    (at -96.85 38.35)
+    (at -96.775 37.725)
     (descr "Resistor, Axial_DIN0204 series, Axial, Horizontal, pin pitch=7.62mm, 0.167W, length*diameter=3.6*1.6mm^2, http://cdn-reichelt.de/documents/datenblatt/B400/1_4W%23YAG.pdf")
     (tags "Resistor Axial_DIN0204 series Axial Horizontal pin pitch 7.62mm 0.167W length 3.6mm diameter 1.6mm")
@@
   )
   (module Capacitor_THT:C_Disc_D4.3mm_W1.9mm_P5.00mm (layer F.Cu)
-    (at -99.575 34.125 270)
+    (at -99.5 35 270)
     (descr "C, Disc series, Radial, pin pitch=5.00mm, , diameter*width=4.3*1.9mm^2, Capacitor, http://www.vishay.com/docs/45233/krseries.pdf")
     (tags "C Disc series Radial pin pitch 5.00mm  diameter 4.3mm width 1.9mm Capacitor")
@@
   (segment (start -118.22537 39.584) (end -121.666 36.14337) (width 1) (layer B.Cu) (net 4))
   (segment (start -121.666 24.892) (end -122.183 24.892) (width 1) (layer B.Cu) (net 4))
-  (segment (start -103.336 35.09) (end -102.362 34.116) (width 1) (layer F.Cu) (net 4))
   (segment (start -105.08 35.09) (end -103.336 35.09) (width 1) (layer F.Cu) (net 4))
   (segment (start -93.695 67.789) (end -93.695 70.104) (width 1) (layer B.Cu) (net 4))
@@
   (segment (start -95.465 52.525) (end -93.375 54.615) (width 1) (layer F.Cu) (net 4))
   (segment (start -99.797 52.525) (end -95.465 52.525) (width 1) (layer F.Cu) (net 4))
-  (segment (start -90.17 40.894) (end -90.17 51.41) (width 1) (layer B.Cu) (net 4))
   (segment (start -90.17 51.41) (end -93.375 54.615) (width 1) (layer B.Cu) (net 4))
   (segment (start -88.725009 54.224991) (end -92.984991 54.224991) (width 1) (layer F.Cu) (net 4))
@@
   (segment (start -88.646 60.706) (end -88.646 55.96807) (width 1) (layer F.Cu) (net 4))
   (segment (start -99.575 37.65) (end -99.575 39.125) (width 1) (layer B.Cu) (net 4))
-  (segment (start -102.362 36.338) (end -99.575 39.125) (width 1) (layer F.Cu) (net 4))
-  (segment (start -102.362 34.116) (end -102.362 36.338) (width 1) (layer F.Cu) (net 4))
-  (segment (start -90.6695 40.3945) (end -90.17 40.894) (width 1) (layer B.Cu) (net 4))
   (segment (start -97.282 24.455) (end -97.282 34.482) (width 1) (layer B.Cu) (net 4))
   (segment (start -99.575 36.775) (end -99.575 37.65) (width 1) (layer B.Cu) (net 4))
-  (segment (start -97.65 34.85) (end -97.65 35.1) (width 1) (layer B.Cu) (net 4))
   (segment (start -97.65 34.85) (end -99.575 36.775) (width 1) (layer B.Cu) (net 4))
   (segment (start -97.282 34.482) (end -97.65 34.85) (width 1) (layer B.Cu) (net 4))
-  (segment (start -97.65 35.1) (end -96.025 36.725) (width 1) (layer B.Cu) (net 4))
-  (segment (start -96.025 36.725) (end -95.025 36.725) (width 1) (layer B.Cu) (net 4))
-  (segment (start -91.3555 40.3945) (end -90.6695 40.3945) (width 1) (layer B.Cu) (net 4))
-  (segment (start -95.025 36.725) (end -91.3555 40.3945) (width 1) (layer B.Cu) (net 4))
   (segment (start -106.174 69.15) (end -119.243 69.15) (width 1) (layer F.Cu) (net 4))
   (segment (start -119.634 57.69) (end -119.634 68.759) (width 1) (layer F.Cu) (net 4))
   (segment (start -119.243 69.15) (end -119.634 68.759) (width 1) (layer F.Cu) (net 4))
   (segment (start -119.634 68.759) (end -119.634 69.596) (width 1) (layer F.Cu) (net 4))
+  (segment (start -97.65 34.85) (end -97.65 35.1) (width 1) (layer B.Cu) (net 4))
+  (segment (start -90.17 40.894) (end -90.17 51.41) (width 1) (layer B.Cu) (net 4))
+  (segment (start -103.237 34.991) (end -103.336 35.09) (width 1) (layer F.Cu) (net 4))
+  (segment (start -102.287 34.991) (end -103.237 34.991) (width 1) (layer F.Cu) (net 4))
+  (segment (start -99.5 37.778) (end -102.287 34.991) (width 1) (layer F.Cu) (net 4))
+  (segment (start -99.5 40) (end -99.5 37.778) (width 1) (layer F.Cu) (net 4))
+  (segment (start -98.606 40.894) (end -99.5 40) (width 1) (layer B.Cu) (net 4))
+  (segment (start -90.17 40.894) (end -98.606 40.894) (width 1) (layer B.Cu) (net 4))
   (segment (start -109.695 4.572) (end -108.689 5.578) (width 1) (layer F.Cu) (net 5))
   (segment (start -109.695 -2.7) (end -109.695 4.572) (width 1) (layer F.Cu) (net 5))
@@
   (segment (start -121.158 10.668) (end -124.206 13.716) (width 1) (layer F.Cu) (net 5))
   (segment (start -117.348 10.668) (end -121.158 10.668) (width 1) (layer F.Cu) (net 5))
-  (segment (start -102.362 39.116) (end -103.886 37.592) (width 1) (layer F.Cu) (net 6))
-  (segment (start -105.042 37.592) (end -105.08 37.63) (width 1) (layer F.Cu) (net 6))
-  (segment (start -103.886 37.592) (end -105.042 37.592) (width 1) (layer F.Cu) (net 6))
+  (segment (start -102.287 38.413) (end -102.287 39.991) (width 1) (layer F.Cu) (net 6))
+  (segment (start -105.08 37.63) (end -105.042 37.592) (width 1) (layer F.Cu) (net 6))
+  (segment (start -103.108 37.592) (end -102.287 38.413) (width 1) (layer F.Cu) (net 6))
+  (segment (start -105.042 37.592) (end -103.108 37.592) (width 1) (layer F.Cu) (net 6))
   (segment (start -96.047 15.6) (end -99.822 19.375) (width 1) (layer F.Cu) (net 7))
   (segment (start -93.45 15.6) (end -96.047 15.6) (width 1) (layer F.Cu) (net 7))
@@
   (segment (start -106.642 40.17) (end -105.08 40.17) (width 1) (layer B.Cu) (net 7))
   (segment (start -111.722 35.09) (end -106.642 40.17) (width 1) (layer B.Cu) (net 7))
-  (segment (start -105.08 40.17) (end -103.848 41.402) (width 1) (layer F.Cu) (net 7))
-  (segment (start -101.372001 41.428001) (end -101.346 41.402) (width 1) (layer F.Cu) (net 7))
-  (segment (start -101.346 41.402) (end -99.314 41.402) (width 1) (layer F.Cu) (net 7))
   (via (at -90.424 63.48) (size 0.8) (drill 0.4) (layers F.Cu B.Cu) (net 7))
   (segment (start -91.674 62.23) (end -90.424 63.48) (width 1) (layer F.Cu) (net 7))
@@
   (segment (start -90.424 63.48) (end -88.626 63.48) (width 1) (layer F.Cu) (net 7))
   (segment (start -88.626 63.48) (end -87.122 61.976) (width 1) (layer F.Cu) (net 7))
-  (segment (start -102.223 41.402) (end -102.223 48.927) (width 1) (layer F.Cu) (net 7))
-  (segment (start -102.223 41.402) (end -101.346 41.402) (width 1) (layer F.Cu) (net 7))
-  (segment (start -103.848 41.402) (end -102.223 41.402) (width 1) (layer F.Cu) (net 7))
   (segment (start -101.165 49.985) (end -99.797 49.985) (width 1) (layer F.Cu) (net 7))
   (segment (start -102.223 48.927) (end -101.165 49.985) (width 1) (layer F.Cu) (net 7))
-  (segment (start -96.85 38.938) (end -96.85 38.35) (width 1) (layer F.Cu) (net 7))
-  (segment (start -99.314 41.402) (end -96.85 38.938) (width 1) (layer F.Cu) (net 7))
+  (segment (start -96.775 40.575) (end -96.775 37.725) (width 1) (layer F.Cu) (net 7))
+  (segment (start -98.675 42.475) (end -96.775 40.575) (width 1) (layer F.Cu) (net 7))
+  (segment (start -105.08 40.17) (end -102.775 42.475) (width 1) (layer F.Cu) (net 7))
+  (segment (start -102.15 42.475) (end -102.15 48.854) (width 1) (layer F.Cu) (net 7))
+  (segment (start -102.15 42.475) (end -98.675 42.475) (width 1) (layer F.Cu) (net 7))
+  (segment (start -102.15 48.854) (end -102.223 48.927) (width 1) (layer F.Cu) (net 7))
+  (segment (start -102.775 42.475) (end -102.15 42.475) (width 1) (layer F.Cu) (net 7))
   (segment (start -114.808 3.048) (end -117.348 3.048) (width 1) (layer F.Cu) (net 8))
   (segment (start -117.348 -4.064) (end -117.348 3.048) (width 1) (layer B.Cu) (net 8))
@@
   (segment (start -90.932 8.627998) (end -90.932 31.942002) (width 1) (layer B.Cu) (net 8))
   (segment (start -90.932 31.942002) (end -93.787998 34.798) (width 1) (layer B.Cu) (net 8))
-  (segment (start -98.806 34.798) (end -99.568 34.036) (width 1) (layer F.Cu) (net 8))
   (segment (start -95.758 34.798) (end -98.806 34.798) (width 1) (layer F.Cu) (net 8))
   (segment (start -106.580001 23.429999) (end -105.08 24.93) (width 1) (layer B.Cu) (net 8))
@@
   (segment (start -91.948 36.576) (end -91.948 37.698) (width 1) (layer F.Cu) (net 13))
   (segment (start -91.771 38.35) (end -91.948 38.527) (width 1) (layer F.Cu) (net 13))
-  (segment (start -89.23 38.35) (end -91.771 38.35) (width 1) (layer F.Cu) (net 13))
   (segment (start -91.948 37.698) (end -91.948 38.527) (width 1) (layer F.Cu) (net 13))
   (segment (start -91.948 38.527) (end -91.948 43.188) (width 1) (layer F.Cu) (net 13))
+  (segment (start -91.921 37.725) (end -91.948 37.698) (width 1) (layer F.Cu) (net 13))
+  (segment (start -89.155 37.725) (end -91.921 37.725) (width 1) (layer F.Cu) (net 13))
   (segment (start -125.025 37.05) (end -125.025 37.649) (width 1) (layer F.Cu) (net 14))
   (segment (start -120.487 32.512) (end -125.025 37.05) (width 1) (layer F.Cu) (net 14))

Commit message: update
Parts:
- moved C2 2.18 mm to (-122.0, 13.6)
- moved C4 2.18 mm to (-122.0, 16.7)
- moved R5 1.49 mm to (-116.0, 2.20)
- moved R4 1.49 mm to (-118.6, 9.82)
Routing:
- net VCC: track 170.9 -> 167.8 mm
- net VIN: track 41.4 -> 43.6 mm
- net GND: track 314.8 -> 315.9 mm

Commit message: update
Parts:
- added G***: LOGO, footprints:moth4, F.Cu at (-88.5, 63.0)
- J10: value Conn_01x04_Female -> Conn_01x05_Female; footprint Connector_PinSocket_2.54mm:PinSocket_1x04_P2.54mm_Vertical -> Connector_PinSocket_2.54mm:PinSocket_1x05_P2.54mm_Vertical
- J3: value Screw_Terminal_01x04 -> Screw_Terminal_01x05; footprint TerminalBlock_Phoenix:TerminalBlock_Phoenix_PT-1,5-4-5.0-H_1x04_P5.00mm_Horizontal -> TerminalBlock_Phoenix:TerminalBlock_Phoenix_PT-1,5-5-5.0-H_1x05_P5.00mm_Horizontal
- moved J10 2.94 mm to (-117.9, 22.1)
- moved R3 2.88 mm to (-121.9, 48.1)
- moved R6 2.88 mm to (-121.9, 50.1)
- moved J5 1.14 mm to (-93.0, 62.1)
- moved U3 0.60 mm to (-113.4, 15.5)
- moved C5 0.53 mm to (-116.9, 36.6)
- moved J3 0.50 mm to (-124.8, 21.6)
- moved J1 0.28 mm to (-124.7, 3.48)
- moved J6 0.20 mm to (-100.0, 19.4)
- moved J11 0.18 mm to (-100.0, 52.5)
Connections:
- J10 pad 1: GND -> VIN
- J10 pad 2: VCC -> GND
- J10 pad 3: D3 -> VCC
- J10 pad 4: D4 -> D3
- J3 pad 1: GND -> VIN
- J3 pad 2: VCC -> GND
- J3 pad 3: D3 -> VCC
- J3 pad 4: D4 -> D3
Routing:
- net GND: track 315.9 -> 350.0 mm
- net VIN: track 43.6 -> 55.2 mm
- net VCC: track 167.8 -> 179.3 mm
- net D5: track 35.3 -> 30.7 mm
- net RST: track 109.5 -> 112.5 mm
- net D3: track 13.2 -> 15.8 mm
- net Net-(D1-Pad1): track 14.0 -> 11.9 mm
- net D4: track 25.6 -> 27.4 mm
- net MOSI: track 54.6 -> 53.4 mm
- net A0: track 34.7 -> 35.7 mm
- net SCK: track 47.1 -> 47.7 mm
- net MISO: track 54.3 -> 54.9 mm
Other:
- board text added: "(M2.5)"
- board text added: "1/GND"
- board text added: "2/MISO"
- board text added: "3V"
- board text added: "9/ANT"
- board text added: "A0"
- board text added: "A4"
- board text added: "A5"
- board text added: "AT1"
- board text added: "D3"
- board text added: "D4"
- board text added: "DTR"
- board text added: "GND"
- board text added: "MISO"
- board text added: "MOSI"
- board text added: "RESET"
- board text added: "RFM95"
- board text added: "RST"
- board text added: "RX"
- board text added: "SCK"
- board text added: "SCL"
- board text added: "SDA"
- board text added: "TX"
- board text added: "VIN"
- board text added: "pvos.org/ mothbot"
- board text added: "ver3"
