File: ver3/dippy.kicad_pcb (KiCad board)
At the start: 2 copper layers, 46.6 x 79.2 mm, 38 parts, among them J1 Screw_Terminal_01x02, J10 Conn_01x05_Female, J2 Screw_Terminal_01x03, J3 Screw_Terminal_01x05, J4 Conn_Coaxial, J5 Conn_02x03_Odd_Even, J6 Conn_01x04_Female, J7 Conn_01x05_Female, J8 Screw_Terminal_01x04, J9 Conn_01x03_Female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

Commit message: update
Parts:
- moved Y1 1.75 mm to (-117.3, 46.5)
- moved G*** 0.85 mm to (-102.0, 62.0), turned to 90 degrees
- moved C5 0.35 mm to (-117.3, 37.9)
- moved R6 0.18 mm to (-122.0, 50.3)
Routing:
- net Net-(U1-Pad10): track 8.92 -> 14.5 mm
- net D8: track 23.9 -> 26.4 mm
- net D7: track 29.7 -> 32.2 mm
- net Net-(U1-Pad9): track 6.53 -> 8.92 mm
- net RST: track 115.1 -> 116.8 mm
- net VCC: track 185.3 -> 186.9 mm
- net D5: track 30.7 -> 29.3 mm, vias 1 -> 0
- net GND: track 336.4 -> 337.8 mm, vias 4 -> 5
- net SCK: track 50.4 -> 51.2 mm
Other:
- board text added: "VER:3"
- board text removed: "ver:3"
