File: ver3/dippy.sch (KiCad schematic (older format))
At the start: 22 parts, among them J1 Conn_01x02_Female, J2 Screw_Terminal_01x03, J3 Screw_Terminal_01x04, J4 Conn_Coaxial, J5 Conn_02x03_Odd_Even, U1 ATmega328P-PU-C, U2 RFM95W-915S2, U3 MCP1700-3302E_SOT23, Y1 Crystal

Commit message: update
Parts:
- added H3, H4: MountingHole, MountingHole:MountingHole_2.7mm_M2.5, symbol Mechanical:MountingHole
Changed lines of the file:
@@
+	1    0    0    -1
+$EndComp
+$Comp
+L Mechanical:MountingHole H3
+U 1 1 5F3B9C3E
+P 6050 2750
+F 0 "H3" H 6150 2796 50  0000 L CNN
+F 1 "MountingHole" H 6150 2705 50  0000 L CNN
+F 2 "MountingHole:MountingHole_2.7mm_M2.5" H 6050 2750 50  0001 C CNN
+F 3 "~" H 6050 2750 50  0001 C CNN
+	1    6050 2750
+	1    0    0    -1
+$EndComp
+$Comp
+L Mechanical:MountingHole H4
+U 1 1 5F3BA0EE
+P 6050 3050
+F 0 "H4" H 6150 3096 50  0000 L CNN
+F 1 "MountingHole" H 6150 3005 50  0000 L CNN
+F 2 "MountingHole:MountingHole_2.7mm_M2.5" H 6050 3050 50  0001 C CNN
+F 3 "~" H 6050 3050 50  0001 C CNN
+	1    6050 3050
 	1    0    0    -1
 $EndComp

Commit message: update
Parts:
- added J6: Screw_Terminal_01x04, TerminalBlock_Phoenix:TerminalBlock_Phoenix_PT-1,5-4-3.5-H_1x04_P3.50mm_Horizontal, symbol Connector:Screw_Terminal_01x04
- added J7: Conn_01x02_Female, Connector_PinSocket_2.54mm:PinSocket_1x02_P2.54mm_Vertical, symbol Connector:Conn_01x02_Female
Connections:
- net A0: now also J2.3 (Pin_3), R2.2; no longer J3.3 (Pin_3), R3.2
- net A1: now also J7.2 (Pin_2); no longer J3.4 (Pin_4)
- net A2: now also J7.1 (Pin_1); no longer J2.2 (Pin_2), R2.2
- net A3: now also R4.2, R5.1
- net A4: now also J6.3 (Pin_3)
- net A5: now also J6.4 (Pin_4); no longer R4.2, R5.1
- net D2: now also U2.14 (DIO0)
- net D3: now also J3.3 (Pin_3); no longer U2.14 (DIO0)
- net D4: now also J3.4 (Pin_4), R3.2
- net GND: now also J6.2 (Pin_2)
- net VCC: now also J2.2 (Pin_2), J6.1 (Pin_1); no longer J2.3 (Pin_3)
Other:
- moved on the sheet: C2, C4, C5, J1, J3, R3, R4, R5, U3

Commit message: update
Parts:
- added D1: LED, LED_THT:LED_D3.0mm, symbol Device:LED
- added R6: 300R, Resistor_THT:R_Axial_DIN0204_L3.6mm_D1.6mm_P5.08mm_Horizontal, symbol Device:R
Connections:
- net D5: now also D1.2 (A)
- net GND: now also R6.2
- new net: D1.1 (K), R6.1
Other:
- moved on the sheet: J7
Changed lines of the file:
@@
 L Connector:Conn_01x02_Female J7
 U 1 1 5F537DB5
-P 5200 4000
-F 0 "J7" H 5228 3976 50  0000 L CNN
-F 1 "Conn_01x02_Female" H 5228 3885 50  0000 L CNN
-F 2 "Connector_PinSocket_2.54mm:PinSocket_1x02_P2.54mm_Vertical" H 5200 4000 50  0001 C CNN
-F 3 "~" H 5200 4000 50  0001 C CNN
-	1    5200 4000
+P 4650 3900
+F 0 "J7" H 4678 3876 50  0000 L CNN
+F 1 "Conn_01x02_Female" H 4678 3785 50  0000 L CNN
+F 2 "Connector_PinSocket_2.54mm:PinSocket_1x02_P2.54mm_Vertical" H 4650 3900 50  0001 C CNN
+F 3 "~" H 4650 3900 50  0001 C CNN
+	1    4650 3900
 	1    0    0    -1
 $EndComp
-Text GLabel 5000 4100 0    50   Input ~ 0
+Text GLabel 4450 4000 0    50   Input ~ 0
 A1
-Text GLabel 5000 4000 0    50   Input ~ 0
+Text GLabel 4450 3900 0    50   Input ~ 0
 A2
+$Comp
+L Device:LED D1
+U 1 1 5F57E191
+P 9800 3900
+F 0 "D1" V 9839 3782 50  0000 R CNN
+F 1 "LED" V 9748 3782 50  0000 R CNN
+F 2 "LED_THT:LED_D3.0mm" H 9800 3900 50  0001 C CNN
+F 3 "~" H 9800 3900 50  0001 C CNN
+	1    9800 3900
+	0    -1   -1   0
+$EndComp
+Text GLabel 9800 3750 0    50   Input ~ 0
+D5
+$Comp
+L power:GND #PWR0124
+U 1 1 5F5807E4
+P 9800 4350
+F 0 "#PWR0124" H 9800 4100 50  0001 C CNN
+F 1 "GND" H 9805 4177 50  0000 C CNN
+F 2 "" H 9800 4350 50  0001 C CNN
+F 3 "" H 9800 4350 50  0001 C CNN
+	1    9800 4350
+	1    0    0    -1
+$EndComp
+$Comp
+L Device:R R6
+U 1 1 5F59A5EA
+P 9800 4200
+F 0 "R6" H 9870 4246 50  0000 L CNN
+F 1 "300R" H 9870 4155 50  0000 L CNN
+F 2 "Resistor_THT:R_Axial_DIN0204_L3.6mm_D1.6mm_P5.08mm_Horizontal" V 9730 4200 50  0001 C CNN
+F 3 "~" H 9800 4200 50  0001 C CNN
+	1    9800 4200
+	1    0    0    -1
+$EndComp
 $EndSCHEMATC

Commit message: update
Connections:
- net RST: now reaches C1.1, J5.5 (Pin_5), R1.2, U1.1 (~RESET~/PC6)
Other:
- moved on the sheet: C1, C2, C3, C4, C5, D1, FTDI1, H1, H2, H3, H4, J1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
