File: ver3/dippy.sch (KiCad schematic (older format))
At the start: 37 parts, among them J1 Screw_Terminal_01x02, J10 Conn_01x04_Female, J11 Conn_01x03_Female, J2 Screw_Terminal_01x03, J3 Screw_Terminal_01x04, J4 Conn_Coaxial, J5 Conn_02x03_Odd_Even, J6 Conn_01x04_Female, J7 Conn_01x03_Female, J8 Screw_Terminal_01x04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

Commit message: update
Parts:
- removed H3, H4: MountingHole, MountingHole:MountingHole_2.7mm_M2.5, symbol Mechanical:MountingHole
- C1, C2, C3, C4, C6: footprint Capacitor_THT:C_Disc_D3.0mm_W1.6mm_P2.50mm -> Capacitor_THT:C_Disc_D4.3mm_W1.9mm_P5.00mm
- D1: footprint LED_THT:LED_D3.0mm -> LED_THT:LED_D5.0mm
- J1: footprint TerminalBlock_Phoenix:TerminalBlock_Phoenix_PT-1,5-2-3.5-H_1x02_P3.50mm_Horizontal -> TerminalBlock_Phoenix:TerminalBlock_Phoenix_PT-1,5-2-5.0-H_1x02_P5.00mm_Horizontal
- J11, J7: footprint Connector_PinHeader_2.54mm:PinHeader_1x03_P2.54mm_Vertical -> Connector_PinSocket_2.54mm:PinSocket_1x03_P2.54mm_Vertical
- J2: footprint TerminalBlock_Phoenix:TerminalBlock_Phoenix_PT-1,5-3-3.5-H_1x03_P3.50mm_Horizontal -> TerminalBlock_Phoenix:TerminalBlock_Phoenix_PT-1,5-3-5.0-H_1x03_P5.00mm_Horizontal
- J3, J8: footprint TerminalBlock_Phoenix:TerminalBlock_Phoenix_PT-1,5-4-3.5-H_1x04_P3.50mm_Horizontal -> TerminalBlock_Phoenix:TerminalBlock_Phoenix_PT-1,5-4-5.0-H_1x04_P5.00mm_Horizontal
- R1, R2, R3, R4, R5, R6, R7, R8: footprint Resistor_THT:R_Axial_DIN0204_L3.6mm_D1.6mm_P5.08mm_Horizontal -> Resistor_THT:R_Axial_DIN0204_L3.6mm_D1.6mm_P7.62mm_Horizontal
Connections:
- net GND: now also SW1.3; no longer SW1.2
- net RST: now also SW1.2; no longer SW1.3
Changed lines of the file:
@@
 F 0 "R1" H 1220 1496 50  0000 L CNN
 F 1 "10K" H 1220 1405 50  0000 L CNN
-F 2 "Resistor_THT:R_Axial_DIN0204_L3.6mm_D1.6mm_P5.08mm_Horizontal" V 1080 1450 50  0001 C CNN
+F 2 "Resistor_THT:R_Axial_DIN0204_L3.6mm_D1.6mm_P7.62mm_Horizontal" V 1080 1450 50  0001 C CNN
 F 3 "~" H 1150 1450 50  0001 C CNN
 	1    1150 1450
@@
 F 0 "C3" H 4765 2846 50  0000 L CNN
 F 1 "0.1u" H 4765 2755 50  0000 L CNN
-F 2 "Capacitor_THT:C_Disc_D3.0mm_W1.6mm_P2.50mm" H 4688 2650 50  0001 C CNN
+F 2 "Capacitor_THT:C_Disc_D4.3mm_W1.9mm_P5.00mm" H 4688 2650 50  0001 C CNN
 F 3 "~" H 4650 2800 50  0001 C CNN
 	1    4650 2800
@@
 F 0 "C1" V 898 2000 50  0000 C CNN
 F 1 "0.1u" V 989 2000 50  0000 C CNN
-F 2 "Capacitor_THT:C_Disc_D3.0mm_W1.6mm_P2.50mm" H 1188 1850 50  0001 C CNN
+F 2 "Capacitor_THT:C_Disc_D4.3mm_W1.9mm_P5.00mm" H 1188 1850 50  0001 C CNN
 F 3 "~" H 1150 2000 50  0001 C CNN
 	1    1150 2000
@@
 F 0 "C2" H 3715 5596 50  0000 L CNN
 F 1 "0.1u" H 3715 5505 50  0000 L CNN
-F 2 "Capacitor_THT:C_Disc_D3.0mm_W1.6mm_P2.50mm" H 3638 5400 50  0001 C CNN
+F 2 "Capacitor_THT:C_Disc_D4.3mm_W1.9mm_P5.00mm" H 3638 5400 50  0001 C CNN
 F 3 "~" H 3600 5550 50  0001 C CNN
 	1    3600 5550
@@
 F 0 "C4" H 4815 5596 50  0000 L CNN
 F 1 "0.1u" H 4815 5505 50  0000 L CNN
-F 2 "Capacitor_THT:C_Disc_D3.0mm_W1.6mm_P2.50mm" H 4738 5400 50  0001 C CNN
+F 2 "Capacitor_THT:C_Disc_D4.3mm_W1.9mm_P5.00mm" H 4738 5400 50  0001 C CNN
 F 3 "~" H 4700 5550 50  0001 C CNN
 	1    4700 5550
@@
 F 0 "J2" H 6730 5642 50  0000 L CNN
 F 1 "Screw_Terminal_01x03" H 6730 5551 50  0001 L CNN
-F 2 "TerminalBlock_Phoenix:TerminalBlock_Phoenix_PT-1,5-3-3.5-H_1x03_P3.50mm_Horizontal" H 6650 5600 50  0001 C CNN
+F 2 "TerminalBlock_Phoenix:TerminalBlock_Phoenix_PT-1,5-3-5.0-H_1x03_P5.00mm_Horizontal" H 6650 5600 50  0001 C CNN
 F 3 "~" H 6650 5600 50  0001 C CNN
 	1    6650 5600
@@
 F 0 "J3" H 6680 4192 50  0000 L CNN
 F 1 "Screw_Terminal_01x04" H 6680 4101 50  0001 L CNN
-F 2 "TerminalBlock_Phoenix:TerminalBlock_Phoenix_PT-1,5-4-3.5-H_1x04_P3.50mm_Horizontal" H 6600 4200 50  0001 C CNN
+F 2 "TerminalBlock_Phoenix:TerminalBlock_Phoenix_PT-1,5-4-5.0-H_1x04_P5.00mm_Horizontal" H 6600 4200 50  0001 C CNN
 F 3 "~" H 6600 4200 50  0001 C CNN
 	1    6600 4200
@@
 F 0 "R2" H 8170 5596 50  0000 L CNN
 F 1 "10K" H 8170 5505 50  0000 L CNN
-F 2 "Resistor_THT:R_Axial_DIN0204_L3.6mm_D1.6mm_P5.08mm_Horizontal" V 8030 5550 50  0001 C CNN
+F 2 "Resistor_THT:R_Axial_DIN0204_L3.6mm_D1.6mm_P7.62mm_Horizontal" V 8030 5550 50  0001 C CNN
 F 3 "~" H 8100 5550 50  0001 C CNN
 	1    8100 5550
@@
 F 0 "R3" H 7870 4296 50  0000 L CNN
 F 1 "10K" H 7870 4205 50  0000 L CNN
-F 2 "Resistor_THT:R_Axial_DIN0204_L3.6mm_D1.6mm_P5.08mm_Horizontal" V 7730 4250 50  0001 C CNN
+F 2 "Resistor_THT:R_Axial_DIN0204_L3.6mm_D1.6mm_P7.62mm_Horizontal" V 7730 4250 50  0001 C CNN
 F 3 "~" H 7800 4250 50  0001 C CNN
 	1    7800 4250
@@
 F 0 "R4" H 9720 1646 50  0000 L CNN
 F 1 "10M" H 9720 1555 50  0000 L CNN
-F 2 "Resistor_THT:R_Axial_DIN0204_L3.6mm_D1.6mm_P5.08mm_Horizontal" V 9580 1600 50  0001 C CNN
+F 2 "Resistor_THT:R_Axial_DIN0204_L3.6mm_D1.6mm_P7.62mm_Horizontal" V 9580 1600 50  0001 C CNN
 F 3 "~" H 9650 1600 50  0001 C CNN
 	1    9650 1600
@@
 F 0 "R5" H 9720 2096 50  0000 L CNN
 F 1 "10M" H 9720 2005 50  0000 L CNN
-F 2 "Resistor_THT:R_Axial_DIN0204_L3.6mm_D1.6mm_P5.08mm_Horizontal" V 9580 2050 50  0001 C CNN
+F 2 "Resistor_THT:R_Axial_DIN0204_L3.6mm_D1.6mm_P7.62mm_Horizontal" V 9580 2050 50  0001 C CNN
 F 3 "~" H 9650 2050 50  0001 C CNN
 	1    9650 2050
@@
 F 3 "~" H 6000 6850 50  0001 C CNN
 	1    6000 6850
-	1    0    0    -1
-$EndComp
-$Comp
-L Mechanical:MountingHole H3
-U 1 1 5F3B9C3E
-P 6000 7200
-F 0 "H3" H 6100 7246 50  0000 L CNN
-F 1 "MountingHole" H 6100 7155 50  0000 L CNN
-F 2 "MountingHole:MountingHole_2.7mm_M2.5" H 6000 7200 50  0001 C CNN
-F 3 "~" H 6000 7200 50  0001 C CNN
-	1    6000 7200
-	1    0    0    -1
-$EndComp
-$Comp
-L Mechanical:MountingHole H4
-U 1 1 5F3BA0EE
-P 6000 7500
-F 0 "H4" H 6100 7546 50  0000 L CNN
-F 1 "MountingHole" H 6100 7455 50  0000 L CNN
-F 2 "MountingHole:MountingHole_2.7mm_M2.5" H 6000 7500 50  0001 C CNN
-F 3 "~" H 6000 7500 50  0001 C CNN
-	1    6000 7500
 	1    0    0    -1
 $EndComp
@@
 F 0 "D1" V 1889 2032 50  0000 R CNN
 F 1 "LED" V 1798 2032 50  0000 R CNN
-F 2 "LED_THT:LED_D3.0mm" H 1850 2150 50  0001 C CNN
+F 2 "LED_THT:LED_D5.0mm" H 1850 2150 50  0001 C CNN
 F 3 "~" H 1850 2150 50  0001 C CNN
 	1    1850 2150
@@
 F 0 "R6" H 1920 2496 50  0000 L CNN
 F 1 "300R" H 1920 2405 50  0000 L CNN
-F 2 "Resistor_THT:R_Axial_DIN0204_L3.6mm_D1.6mm_P5.08mm_Horizontal" V 1780 2450 50  0001 C CNN
+F 2 "Resistor_THT:R_Axial_DIN0204_L3.6mm_D1.6mm_P7.62mm_Horizontal" V 1780 2450 50  0001 C CNN
 F 3 "~" H 1850 2450 50  0001 C CNN
 	1    1850 2450
@@
 F 0 "J7" H 1628 6976 50  0000 L CNN
 F 1 "Conn_01x03_Female" H 1628 6885 50  0001 L CNN
-F 2 "Connector_PinHeader_2.54mm:PinHeader_1x03_P2.54mm_Vertical" H 1600 6950 50  0001 C CNN
+F 2 "Connector_PinSocket_2.54mm:PinSocket_1x03_P2.54mm_Vertical" H 1600 6950 50  0001 C CNN
 F 3 "~" H 1600 6950 50  0001 C CNN
 	1    1600 6950
@@
 Text GLabel 4750 1700 0    50   Input ~ 0
 RST
-Wire Wire Line
-	4750 1700 4750 1900
-Wire Wire Line
-	5150 1700 5150 1900
 $Comp
 L power:GND #PWR0128
@@
 	1    0    0    -1
 $EndComp
-Connection ~ 5150 1900
 $Comp
 L Connector:Conn_01x03_Female J9
@@
 F 0 "R7" H 10670 3646 50  0000 L CNN
 F 1 "R" H 10670 3555 50  0000 L CNN
-F 2 "Resistor_THT:R_Axial_DIN0204_L3.6mm_D1.6mm_P5.08mm_Horizontal" V 10530 3600 50  0001 C CNN
+F 2 "Resistor_THT:R_Axial_DIN0204_L3.6mm_D1.6mm_P7.62mm_Horizontal" V 10530 3600 50  0001 C CNN
 F 3 "~" H 10600 3600 50  0001 C CNN
 	1    10600 3600
@@
 F 0 "R8" H 10870 3646 50  0000 L CNN
 F 1 "R" H 10870 3555 50  0000 L CNN
-F 2 "Resistor_THT:R_Axial_DIN0204_L3.6mm_D1.6mm_P5.08mm_Horizontal" V 10730 3600 50  0001 C CNN
+F 2 "Resistor_THT:R_Axial_DIN0204_L3.6mm_D1.6mm_P7.62mm_Horizontal" V 10730 3600 50  0001 C CNN
 F 3 "~" H 10800 3600 50  0001 C CNN
 	1    10800 3600
@@
 F 0 "J8" H 10118 3175 50  0000 C CNN
 F 1 "Screw_Terminal_01x04" H 10118 3266 50  0001 C CNN
-F 2 "TerminalBlock_Phoenix:TerminalBlock_Phoenix_PT-1,5-4-3.5-H_1x04_P3.50mm_Horizontal" H 10200 3600 50  0001 C CNN
+F 2 "TerminalBlock_Phoenix:TerminalBlock_Phoenix_PT-1,5-4-5.0-H_1x04_P5.00mm_Horizontal" H 10200 3600 50  0001 C CNN
 F 3 "~" H 10200 3600 50  0001 C CNN
 	1    10200 3600
@@
 F 0 "J1" H 2868 5175 50  0000 C CNN
 F 1 "Screw_Terminal_01x02" H 2868 5266 50  0000 C CNN
-F 2 "TerminalBlock_Phoenix:TerminalBlock_Phoenix_PT-1,5-2-3.5-H_1x02_P3.50mm_Horizontal" H 2950 5500 50  0001 C CNN
+F 2 "TerminalBlock_Phoenix:TerminalBlock_Phoenix_PT-1,5-2-5.0-H_1x02_P5.00mm_Horizontal" H 2950 5500 50  0001 C CNN
 F 3 "~" H 2950 5500 50  0001 C CNN
 	1    2950 5500
@@
 F 0 "J11" H 7628 5580 50  0000 L CNN
 F 1 "Conn_01x03_Female" H 7628 5535 50  0001 L CNN
-F 2 "Connector_PinHeader_2.54mm:PinHeader_1x03_P2.54mm_Vertical" H 7600 5600 50  0001 C CNN
+F 2 "Connector_PinSocket_2.54mm:PinSocket_1x03_P2.54mm_Vertical" H 7600 5600 50  0001 C CNN
 F 3 "~" H 7600 5600 50  0001 C CNN
 	1    7600 5600
@@
 F 0 "C6" H 9100 2100 50  0000 L CNN
 F 1 "0.1uF" H 9000 2000 50  0000 L CNN
-F 2 "Capacitor_THT:C_Disc_D3.0mm_W1.6mm_P2.50mm" H 9388 1900 50  0001 C CNN
+F 2 "Capacitor_THT:C_Disc_D4.3mm_W1.9mm_P5.00mm" H 9388 1900 50  0001 C CNN
 F 3 "~" H 9350 2050 50  0001 C CNN
 	1    9350 2050
@@
 Text Notes 4800 1350 0    118  ~ 0
 NEEDS\nREVIEW
+Wire Wire Line
+	5150 1700 5150 1600
+Wire Wire Line
+	5150 1600 4750 1600
+Wire Wire Line
+	4750 1600 4750 1700
+Wire Wire Line
+	5150 1900 5150 1800
+Wire Wire Line
+	5150 1800 4750 1800
+Wire Wire Line
+	4750 1800 4750 1900
+Connection ~ 5150 1900
 $EndSCHEMATC

Commit message: update
Parts:
- added H3, H4: MountingHole, MountingHole:MountingHole_2.7mm_M2.5, symbol Mechanical:MountingHole
Changed lines of the file:
@@
 	4750 1800 4750 1900
 Connection ~ 5150 1900
+$Comp
+L Mechanical:MountingHole H4
+U 1 1 5F3BA0EE
+P 6000 7500
+F 0 "H4" H 6100 7546 50  0000 L CNN
+F 1 "MountingHole" H 6100 7455 50  0000 L CNN
+F 2 "MountingHole:MountingHole_2.7mm_M2.5" H 6000 7500 50  0001 C CNN
+F 3 "~" H 6000 7500 50  0001 C CNN
+	1    6000 7500
+	1    0    0    -1
+$EndComp
+$Comp
+L Mechanical:MountingHole H3
+U 1 1 5F3B9C3E
+P 6000 7200
+F 0 "H3" H 6100 7246 50  0000 L CNN
+F 1 "MountingHole" H 6100 7155 50  0000 L CNN
+F 2 "MountingHole:MountingHole_2.7mm_M2.5" H 6000 7200 50  0001 C CNN
+F 3 "~" H 6000 7200 50  0001 C CNN
+	1    6000 7200
+	1    0    0    -1
+$EndComp
 $EndSCHEMATC

Commit message: update
Parts:
- removed J10: Conn_01x04_Female, Connector_PinSocket_2.54mm:PinSocket_1x04_P2.54mm_Vertical, symbol Connector:Conn_01x04_Female
- removed J3: Screw_Terminal_01x04, TerminalBlock_Phoenix:TerminalBlock_Phoenix_PT-1,5-4-5.0-H_1x04_P5.00mm_Horizontal, symbol Connector:Screw_Terminal_01x04
- added J10: Conn_01x05_Female, Connector_PinSocket_2.54mm:PinSocket_1x05_P2.54mm_Vertical, symbol Connector:Conn_01x05_Female
- added J3: Screw_Terminal_01x05, TerminalBlock_Phoenix:TerminalBlock_Phoenix_PT-1,5-5-5.0-H_1x05_P5.00mm_Horizontal, symbol Connector:Screw_Terminal_01x05
Connections:
- net D3: now also J10.4 (Pin_4), J3.4 (Pin_4)
- net D4: now also J10.5 (Pin_5), J3.5 (Pin_5)
- net GND: now also J10.2 (Pin_2), J3.2 (Pin_2)
- net VCC: now also J10.3 (Pin_3), J3.3 (Pin_3)
- net VIN: now also J10.1 (Pin_1), J3.1 (Pin_1)
Changed lines of the file:
@@
-$EndComp
-$Comp
-L Connector:Screw_Terminal_01x04 J3
-U 1 1 5F312484
-P 6600 4200
-F 0 "J3" H 6680 4192 50  0000 L CNN
-F 1 "Screw_Terminal_01x04" H 6680 4101 50  0001 L CNN
-F 2 "TerminalBlock_Phoenix:TerminalBlock_Phoenix_PT-1,5-4-5.0-H_1x04_P5.00mm_Horizontal" H 6600 4200 50  0001 C CNN
-F 3 "~" H 6600 4200 50  0001 C CNN
-	1    6600 4200
-	1    0    0    -1
 $EndComp
 $Comp
@@
 L power:GND #PWR0116
 U 1 1 5F33656E
-P 6400 4100
-F 0 "#PWR0116" H 6400 3850 50  0001 C CNN
-F 1 "GND" H 6405 3927 50  0000 C CNN
-F 2 "" H 6400 4100 50  0001 C CNN
-F 3 "" H 6400 4100 50  0001 C CNN
-	1    6400 4100
-	-1   0    0    1
+P 5850 4100
+F 0 "#PWR0116" H 5850 3850 50  0001 C CNN
+F 1 "GND" H 5855 3927 50  0000 C CNN
+F 2 "" H 5850 4100 50  0001 C CNN
+F 3 "" H 5850 4100 50  0001 C CNN
+	1    5850 4100
+	1    0    0    -1
 $EndComp
 Text GLabel 3600 4900 0    50   Input ~ 0
@@
 	1150 1700 2850 1700
 $Comp
-L Connector:Conn_01x04_Female J10
-U 1 1 5F7A4B06
-P 7300 4200
-F 0 "J10" H 7328 4130 50  0000 L CNN
-F 1 "Conn_01x04_Female" H 7328 4085 50  0001 L CNN
-F 2 "Connector_PinSocket_2.54mm:PinSocket_1x04_P2.54mm_Vertical" H 7300 4200 50  0001 C CNN
-F 3 "~" H 7300 4200 50  0001 C CNN
-	1    7300 4200
-	1    0    0    -1
-$EndComp
-$Comp
 L power:GND #PWR0133
 U 1 1 5F7B712B
-P 7100 4100
-F 0 "#PWR0133" H 7100 3850 50  0001 C CNN
-F 1 "GND" H 7105 3927 50  0000 C CNN
-F 2 "" H 7100 4100 50  0001 C CNN
-F 3 "" H 7100 4100 50  0001 C CNN
-	1    7100 4100
-	-1   0    0    1
+P 6800 4100
+F 0 "#PWR0133" H 6800 3850 50  0001 C CNN
+F 1 "GND" H 6805 3927 50  0000 C CNN
+F 2 "" H 6800 4100 50  0001 C CNN
+F 3 "" H 6800 4100 50  0001 C CNN
+	1    6800 4100
+	1    0    0    -1
 $EndComp
 $Comp
@@
 	1    0    0    -1
 $EndComp
+$Comp
+L Connector:Conn_01x05_Female J10
+U 1 1 5F890CA8
+P 7300 4200
+F 0 "J10" H 7328 4180 50  0000 L CNN
+F 1 "Conn_01x05_Female" H 7328 4135 50  0001 L CNN
+F 2 "Connector_PinSocket_2.54mm:PinSocket_1x05_P2.54mm_Vertical" H 7300 4200 50  0001 C CNN
+F 3 "~" H 7300 4200 50  0001 C CNN
+	1    7300 4200
+	1    0    0    -1
+$EndComp
+$Comp
+L Connector:Screw_Terminal_01x05 J3
+U 1 1 5F89274F
+P 6600 4200
+F 0 "J3" H 6680 4196 50  0000 L CNN
+F 1 "Screw_Terminal_01x05" H 6680 4151 50  0001 L CNN
+F 2 "TerminalBlock_Phoenix:TerminalBlock_Phoenix_PT-1,5-5-5.0-H_1x05_P5.00mm_Horizontal" H 6600 4200 50  0001 C CNN
+F 3 "~" H 6600 4200 50  0001 C CNN
+	1    6600 4200
+	1    0    0    -1
+$EndComp
+Wire Wire Line
+	6400 4100 5850 4100
+Wire Wire Line
+	7100 4100 6800 4100
+Text GLabel 6400 4000 0    50   Input ~ 0
+VIN
+Text GLabel 7100 4000 0    50   Input ~ 0
+VIN
 $EndSCHEMATC
