File: ver1/dippy.kicad_pcb (KiCad board)
At the start: 2 copper layers, 31.7 x 69.7 mm, 29 parts, among them J1 Conn_01x02_Female, J2 Screw_Terminal_01x03, J3 Screw_Terminal_01x04, J4 Conn_Coaxial, J5 Conn_02x03_Odd_Even, J6 Screw_Terminal_01x04, J7 Conn_01x02_Female, U1 ATmega328P-PU-C, U2 RFM95W-915S2, U3 MCP1700-3302E_TO92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

Commit message: update
Parts:
- added G***: LOGO, footprints:moth4, F.Cu at (136.9, 111.3)
Other:
- board text added: "ver 1"
- board text removed: "ver 0.1"

Commit message: update
Parts:
- removed G***: LOGO, footprints:moth4
- added J8: Conn_01x04_Female, Connector_JST:JST_SH_SM04B-SRSS-TB_1x04-1MP_P1.00mm_Horizontal, F.Cu at (142.6, 89.3)
- added J9: Conn_01x03_Female, Connector_PinSocket_2.54mm:PinSocket_1x03_P2.54mm_Vertical, F.Cu at (132.5, 64.9)
- added SW1: SW_Push_Dual, Button_Switch_SMD:SW_Push_1P1T_NO_CK_KMR2, F.Cu at (144.0, 79.5)
- J6: value Screw_Terminal_01x04 -> Conn_01x04_Female; footprint TerminalBlock_Phoenix:TerminalBlock_Phoenix_PT-1,5-4-3.5-H_1x04_P3.50mm_Horizontal -> Connector_PinSocket_2.54mm:PinSocket_1x04_P2.54mm_Vertical
- J7: value Conn_01x02_Female -> Conn_01x03_Female; footprint Connector_PinSocket_2.54mm:PinSocket_1x02_P2.54mm_Vertical -> Connector_PinHeader_2.54mm:PinHeader_1x03_P2.54mm_Vertical
- moved J6 10.9 mm to (137.0, 80.8), turned to 0 degrees
- moved FTDI1 5.89 mm to (123.7, 60.7)
- moved J7 0.56 mm to (130.3, 87.0)
Routing:
- net GND: track 211.0 -> 226.1 mm, vias 9 -> 10
- net A5: track 10.7 -> 20.6 mm, vias 0 -> 1
- net RST: track 67.7 -> 76.1 mm, vias 1 -> 3
- net RX0: track 18.3 -> 10.8 mm
- net A4: track 10.2 -> 17.0 mm, vias 0 -> 1
- net Net-(C1-Pad2): track 7.89 -> 3.09 mm
- net TX0: track 22.7 -> 18.9 mm
- net A3: track 24.3 -> 27.7 mm, vias 2 -> 1
- net VIN: track 35.0 -> 32.2 mm
- net VCC: track 142.5 -> 144.0 mm, vias 2 -> 3
Other:
- board size 31.7 x 69.7 mm -> 31.7 x 73.7 mm
- board text added: "A4"
- board text added: "A5"
- board text added: "FTDI"
- board text added: "GND"
- board text added: "RESET"
- board text added: "qwiic"
- board text removed: "SCL"
- board text removed: "SDA"

Commit message: update
Parts:
- moved SW1 1.27 mm to (144.0, 80.8)
Routing:
- net RX0: track 10.8 -> 30.0 mm, vias 0 -> 1
- net GND: track 226.1 -> 243.7 mm
- net VIN: track 32.2 -> 46.1 mm, vias 0 -> 2
- net VCC: track 144.0 -> 154.2 mm
- net Net-(C1-Pad2): track 3.09 -> 13.2 mm
- net TX0: track 18.9 -> 28.9 mm
- net RST: track 76.1 -> 77.4 mm

Commit message: update
Parts:
- added R7: R, Resistor_THT:R_Axial_DIN0204_L3.6mm_D1.6mm_P2.54mm_Vertical, F.Cu at (142.4, 83.9)
- added R8: R, Resistor_THT:R_Axial_DIN0204_L3.6mm_D1.6mm_P2.54mm_Vertical, F.Cu at (139.7, 77.6)
- moved SW1 1.14 mm to (144.0, 79.6)
- moved J6 0.13 mm to (136.9, 80.8)
Routing:
- net A5: track 20.6 -> 28.3 mm, vias 1 -> 0
- net A4: track 17.0 -> 21.6 mm
- net VCC: track 154.2 -> 152.8 mm, vias 3 -> 5
- net RST: track 77.4 -> 76.2 mm
- net GND: track 243.7 -> 243.4 mm, vias 10 -> 11
- net A3: track 27.7 -> 27.4 mm, vias 1 -> 0
Other:
- board text added: "DC-DC"
