File: ver1/dippy.sch (KiCad schematic (older format))
At the start: 29 parts, among them J1 Conn_01x02_Female, J2 Screw_Terminal_01x03, J3 Screw_Terminal_01x04, J4 Conn_Coaxial, J5 Conn_02x03_Odd_Even, J6 Screw_Terminal_01x04, J7 Conn_01x02_Female, U1 ATmega328P-PU-C, U2 RFM95W-915S2, U3 MCP1700-3302E_TO92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

Commit message: update
Parts:
- removed U3: MCP1700-3302E_TO92, Package_TO_SOT_THT:TO-92_Inline, symbol mcp1700:MCP1700-3302E_TO92
- added U3: MCP1700-3302E_TO92, Package_TO_SOT_THT:TO-92_Inline, symbol Regulator_Linear:MCP1700-3302E_TO92
Connections:
- net GND: now also U3.1 (GND)
- net VCC: now also U3.3 (VO)
- net VIN: now also U3.2 (VI)
Changed lines of the file:
@@
 $EndComp
 $Comp
-L mcp1700:MCP1700-3302E_TO92 U3
-U 1 1 5F6A0624
+L Regulator_Linear:MCP1700-3302E_TO92 U3
+U 1 1 5F67A451
 P 3350 5450
 F 0 "U3" H 3350 5208 50  0000 C CNN

Commit message: update
Parts:
- removed J6: Screw_Terminal_01x04, TerminalBlock_Phoenix:TerminalBlock_Phoenix_PT-1,5-4-3.5-H_1x04_P3.50mm_Horizontal, symbol Connector:Screw_Terminal_01x04
- removed J7: Conn_01x02_Female, Connector_PinSocket_2.54mm:PinSocket_1x02_P2.54mm_Vertical, symbol Connector:Conn_01x02_Female
- added J6: Conn_01x04_Female, Connector_PinSocket_2.54mm:PinSocket_1x04_P2.54mm_Vertical, symbol Connector:Conn_01x04_Female
- added J7: Conn_01x03_Female, Connector_PinHeader_2.54mm:PinHeader_1x03_P2.54mm_Vertical, symbol Connector:Conn_01x03_Female
- added J8: Conn_01x04_Female, Connector_JST:JST_SH_SM04B-SRSS-TB_1x04-1MP_P1.00mm_Horizontal, symbol Connector:Conn_01x04_Female
- added J9: Conn_01x03_Female, Connector_PinSocket_2.54mm:PinSocket_1x03_P2.54mm_Vertical, symbol Connector:Conn_01x03_Female
- added SW1: SW_Push_Dual, Button_Switch_SMD:SW_Push_1P1T_NO_CK_KMR2, symbol Switch:SW_Push_Dual
Connections:
- net A1: now also J7.2 (Pin_2)
- net A2: now also J7.1 (Pin_1)
- net A4: now also J6.3 (Pin_3), J8.1 (Pin_1)
- net A5: now also J6.4 (Pin_4), J8.2 (Pin_2)
- net GND: now also J6.2 (Pin_2), J7.3 (Pin_3), J8.4 (Pin_4), J9.2 (Pin_2), SW1.2, SW1.4
- net RST: now also SW1.1, SW1.3
- net VCC: now also J6.1 (Pin_1), J8.3 (Pin_3), J9.3 (Pin_3)
- net VIN: now also J9.1 (Pin_1)
Other:
- note added: "5) I2C / Gen purpose"
- note added: "6) DHT22 / SHT10 / UART"
- note removed: "5) Software Serial"
- note removed: "6) DHT22 or SHT10"
Changed lines of the file:
@@
 	1    0    0    -1
 $EndComp
-Text GLabel 9650 3750 0    50   Input ~ 0
+Text GLabel 9350 3750 0    50   Input ~ 0
 A5
-Text GLabel 9650 3650 0    50   Input ~ 0
+Text GLabel 9350 3650 0    50   Input ~ 0
 A4
 $Comp
 L power:GND #PWR0122
 U 1 1 5F44B89B
-P 9300 3550
-F 0 "#PWR0122" H 9300 3300 50  0001 C CNN
-F 1 "GND" H 9305 3377 50  0000 C CNN
-F 2 "" H 9300 3550 50  0001 C CNN
-F 3 "" H 9300 3550 50  0001 C CNN
-	1    9300 3550
+P 9000 3550
+F 0 "#PWR0122" H 9000 3300 50  0001 C CNN
+F 1 "GND" H 9005 3377 50  0000 C CNN
+F 2 "" H 9000 3550 50  0001 C CNN
+F 3 "" H 9000 3550 50  0001 C CNN
+	1    9000 3550
 	1    0    0    -1
 $EndComp
@@
 L power:VCC #PWR0123
 U 1 1 5F44D61B
-P 9650 3450
-F 0 "#PWR0123" H 9650 3300 50  0001 C CNN
-F 1 "VCC" H 9667 3623 50  0000 C CNN
-F 2 "" H 9650 3450 50  0001 C CNN
-F 3 "" H 9650 3450 50  0001 C CNN
-	1    9650 3450
-	1    0    0    -1
-$EndComp
-$Comp
-L Connector:Screw_Terminal_01x04 J6
-U 1 1 5F452A97
-P 9850 3550
-F 0 "J6" H 9930 3542 50  0000 L CNN
-F 1 "Screw_Terminal_01x04" H 9930 3451 50  0000 L CNN
-F 2 "TerminalBlock_Phoenix:TerminalBlock_Phoenix_PT-1,5-4-3.5-H_1x04_P3.50mm_Horizontal" H 9850 3550 50  0001 C CNN
-F 3 "~" H 9850 3550 50  0001 C CNN
-	1    9850 3550
-	1    0    0    -1
-$EndComp
-Wire Wire Line
-	9650 3550 9300 3550
+P 9350 3450
+F 0 "#PWR0123" H 9350 3300 50  0001 C CNN
+F 1 "VCC" H 9367 3623 50  0000 C CNN
+F 2 "" H 9350 3450 50  0001 C CNN
+F 3 "" H 9350 3450 50  0001 C CNN
+	1    9350 3450
+	1    0    0    -1
+$EndComp
+Wire Wire Line
+	9350 3550 9000 3550
 Text GLabel 7750 5750 0    50   Input ~ 0
 A0
@@
 Wire Notes Line
 	800  600  11050 600
-Text Notes 9050 3050 0    118  ~ 0
-5) Software Serial
+Text Notes 8900 3050 0    118  ~ 0
+5) I2C / Gen purpose
 Text Notes 6050 3600 0    118  ~ 0
-6) DHT22 or SHT10
+6) DHT22 / SHT10 / UART
 Wire Notes Line
 	5500 4600 8750 4600
 Wire Notes Line
 	8750 4050 11050 4050
-Text GLabel 1200 7100 0    50   Input ~ 0
+Text GLabel 1400 6850 0    50   Input ~ 0
 A2
-Text GLabel 1200 7200 0    50   Input ~ 0
+Text GLabel 1400 6950 0    50   Input ~ 0
 A1
-$Comp
-L Connector:Conn_01x02_Female J7
-U 1 1 5F537DB5
-P 1400 7100
-F 0 "J7" H 1428 7076 50  0000 L CNN
-F 1 "Conn_01x02_Female" H 1428 6985 50  0000 L CNN
-F 2 "Connector_PinSocket_2.54mm:PinSocket_1x02_P2.54mm_Vertical" H 1400 7100 50  0001 C CNN
-F 3 "~" H 1400 7100 50  0001 C CNN
-	1    1400 7100
-	1    0    0    -1
-$EndComp
 Text GLabel 9650 5000 0    50   Input ~ 0
 MISO
@@
 	1    0    0    1
 $EndComp
+$Comp
+L Connector:Conn_01x04_Female J6
+U 1 1 5F682487
+P 9550 3550
+F 0 "J6" H 9578 3526 50  0000 L CNN
+F 1 "Conn_01x04_Female" V 9750 3200 50  0000 L CNN
+F 2 "Connector_PinSocket_2.54mm:PinSocket_1x04_P2.54mm_Vertical" H 9550 3550 50  0001 C CNN
+F 3 "~" H 9550 3550 50  0001 C CNN
+	1    9550 3550
+	1    0    0    -1
+$EndComp
+$Comp
+L Connector:Conn_01x04_Female J8
+U 1 1 5F688ADE
+P 10650 3500
+F 0 "J8" H 10678 3476 50  0000 L CNN
+F 1 "Conn_01x04_Female" V 10850 3100 50  0000 L CNN
+F 2 "Connector_JST:JST_SH_SM04B-SRSS-TB_1x04-1MP_P1.00mm_Horizontal" H 10650 3500 50  0001 C CNN
+F 3 "~" H 10650 3500 50  0001 C CNN
+	1    10650 3500
+	1    0    0    -1
+$EndComp
+$Comp
+L power:GND #PWR0125
+U 1 1 5F6942B2
+P 10450 3700
+F 0 "#PWR0125" H 10450 3450 50  0001 C CNN
+F 1 "GND" H 10455 3527 50  0000 C CNN
+F 2 "" H 10450 3700 50  0001 C CNN
+F 3 "" H 10450 3700 50  0001 C CNN
+	1    10450 3700
+	1    0    0    -1
+$EndComp
+$Comp
+L power:VCC #PWR0126
+U 1 1 5F6869FA
+P 10150 3600
+F 0 "#PWR0126" H 10150 3450 50  0001 C CNN
+F 1 "VCC" H 10167 3773 50  0000 C CNN
+F 2 "" H 10150 3600 50  0001 C CNN
+F 3 "" H 10150 3600 50  0001 C CNN
+	1    10150 3600
+	1    0    0    -1
+$EndComp
+Wire Wire Line
+	10450 3600 10150 3600
+Text GLabel 10450 3400 0    50   Input ~ 0
+A4
+Text GLabel 10450 3500 0    50   Input ~ 0
+A5
+$Comp
+L Connector:Conn_01x03_Female J7
+U 1 1 5F693D55
+P 1600 6950
+F 0 "J7" H 1628 6976 50  0000 L CNN
+F 1 "Conn_01x03_Female" H 1628 6885 50  0000 L CNN
+F 2 "Connector_PinHeader_2.54mm:PinHeader_1x03_P2.54mm_Vertical" H 1600 6950 50  0001 C CNN
+F 3 "~" H 1600 6950 50  0001 C CNN
+	1    1600 6950
+	1    0    0    -1
+$EndComp
+$Comp
+L power:GND #PWR0127
+U 1 1 5F694F04
+P 1400 7050
+F 0 "#PWR0127" H 1400 6800 50  0001 C CNN
+F 1 "GND" H 1405 6877 50  0000 C CNN
+F 2 "" H 1400 7050 50  0001 C CNN
+F 3 "" H 1400 7050 50  0001 C CNN
+	1    1400 7050
+	1    0    0    -1
+$EndComp
+$Comp
+L Switch:SW_Push_Dual SW1
+U 1 1 5F6B37D1
+P -1200 1050
+F 0 "SW1" H -1200 1335 50  0000 C CNN
+F 1 "SW_Push_Dual" H -1200 1244 50  0000 C CNN
+F 2 "Button_Switch_SMD:SW_Push_1P1T_NO_CK_KMR2" H -1200 1250 50  0001 C CNN
+F 3 "~" H -1200 1250 50  0001 C CNN
+	1    -1200 1050
+	1    0    0    -1
+$EndComp
+Text GLabel -1400 1050 0    50   Input ~ 0
+RST
+Wire Wire Line
+	-1400 1050 -1400 1250
+Wire Wire Line
+	-1000 1050 -1000 1250
+$Comp
+L power:GND #PWR0128
+U 1 1 5F6BD020
+P -1000 1250
+F 0 "#PWR0128" H -1000 1000 50  0001 C CNN
+F 1 "GND" H -995 1077 50  0000 C CNN
+F 2 "" H -1000 1250 50  0001 C CNN
+F 3 "" H -1000 1250 50  0001 C CNN
+	1    -1000 1250
+	1    0    0    -1
+$EndComp
+Connection ~ -1000 1250
+$Comp
+L Connector:Conn_01x03_Female J9
+U 1 1 5F6DC6E3
+P -1300 2800
+F 0 "J9" H -1272 2826 50  0000 L CNN
+F 1 "Conn_01x03_Female" H -1272 2735 50  0000 L CNN
+F 2 "Connector_PinSocket_2.54mm:PinSocket_1x03_P2.54mm_Vertical" H -1300 2800 50  0001 C CNN
+F 3 "~" H -1300 2800 50  0001 C CNN
+	1    -1300 2800
+	1    0    0    -1
+$EndComp
+Text GLabel -1500 2700 0    50   Input ~ 0
+VIN
+$Comp
+L power:GND #PWR0129
+U 1 1 5F6E2E0D
+P -1600 3100
+F 0 "#PWR0129" H -1600 2850 50  0001 C CNN
+F 1 "GND" H -1595 2927 50  0000 C CNN
+F 2 "" H -1600 3100 50  0001 C CNN
+F 3 "" H -1600 3100 50  0001 C CNN
+	1    -1600 3100
+	1    0    0    -1
+$EndComp
+$Comp
+L power:VCC #PWR0130
+U 1 1 5F6E4957
+P -1950 2900
+F 0 "#PWR0130" H -1950 2750 50  0001 C CNN
+F 1 "VCC" H -1933 3073 50  0000 C CNN
+F 2 "" H -1950 2900 50  0001 C CNN
+F 3 "" H -1950 2900 50  0001 C CNN
+	1    -1950 2900
+	1    0    0    -1
+$EndComp
+Wire Wire Line
+	-1500 2800 -1600 2800
+Wire Wire Line
+	-1500 2900 -1950 2900
+Wire Wire Line
+	-1600 2800 -1600 3100
 $EndSCHEMATC

Commit message: update
Parts:
- added R7, R8: R, Resistor_THT:R_Axial_DIN0204_L3.6mm_D1.6mm_P2.54mm_Vertical, symbol Device:R
Connections:
- net A4: now also R7.2
- net A5: now also R8.2
- net VCC: now also R7.1, R8.1
Other:
- moved on the sheet: J6, J8
Changed lines of the file:
@@
 	1    0    0    -1
 $EndComp
-Text GLabel 9350 3750 0    50   Input ~ 0
+Text GLabel 9250 3750 0    50   Input ~ 0
 A5
-Text GLabel 9350 3650 0    50   Input ~ 0
+Text GLabel 9250 3650 0    50   Input ~ 0
 A4
 $Comp
 L power:GND #PWR0122
 U 1 1 5F44B89B
-P 9000 3550
-F 0 "#PWR0122" H 9000 3300 50  0001 C CNN
-F 1 "GND" H 9005 3377 50  0000 C CNN
-F 2 "" H 9000 3550 50  0001 C CNN
-F 3 "" H 9000 3550 50  0001 C CNN
-	1    9000 3550
+P 8900 3550
+F 0 "#PWR0122" H 8900 3300 50  0001 C CNN
+F 1 "GND" H 8905 3377 50  0000 C CNN
+F 2 "" H 8900 3550 50  0001 C CNN
+F 3 "" H 8900 3550 50  0001 C CNN
+	1    8900 3550
 	1    0    0    -1
 $EndComp
@@
 L power:VCC #PWR0123
 U 1 1 5F44D61B
-P 9350 3450
-F 0 "#PWR0123" H 9350 3300 50  0001 C CNN
-F 1 "VCC" H 9367 3623 50  0000 C CNN
-F 2 "" H 9350 3450 50  0001 C CNN
-F 3 "" H 9350 3450 50  0001 C CNN
-	1    9350 3450
-	1    0    0    -1
-$EndComp
-Wire Wire Line
-	9350 3550 9000 3550
+P 9250 3450
+F 0 "#PWR0123" H 9250 3300 50  0001 C CNN
+F 1 "VCC" H 9267 3623 50  0000 C CNN
+F 2 "" H 9250 3450 50  0001 C CNN
+F 3 "" H 9250 3450 50  0001 C CNN
+	1    9250 3450
+	1    0    0    -1
+$EndComp
+Wire Wire Line
+	9250 3550 8900 3550
 Text GLabel 7750 5750 0    50   Input ~ 0
 A0
@@
 Text Notes 8900 3050 0    118  ~ 0
 5) I2C / Gen purpose
-Text Notes 6050 3600 0    118  ~ 0
+Text Notes 5700 3650 0    118  ~ 0
 6) DHT22 / SHT10 / UART
 Wire Notes Line
@@
 L Connector:Conn_01x04_Female J6
 U 1 1 5F682487
-P 9550 3550
-F 0 "J6" H 9578 3526 50  0000 L CNN
-F 1 "Conn_01x04_Female" V 9750 3200 50  0000 L CNN
-F 2 "Connector_PinSocket_2.54mm:PinSocket_1x04_P2.54mm_Vertical" H 9550 3550 50  0001 C CNN
-F 3 "~" H 9550 3550 50  0001 C CNN
-	1    9550 3550
+P 9450 3550
+F 0 "J6" H 9478 3526 50  0000 L CNN
+F 1 "Conn_01x04_Female" V 9650 3200 50  0000 L CNN
+F 2 "Connector_PinSocket_2.54mm:PinSocket_1x04_P2.54mm_Vertical" H 9450 3550 50  0001 C CNN
+F 3 "~" H 9450 3550 50  0001 C CNN
+	1    9450 3550
 	1    0    0    -1
 $EndComp
@@
 L Connector:Conn_01x04_Female J8
 U 1 1 5F688ADE
-P 10650 3500
-F 0 "J8" H 10678 3476 50  0000 L CNN
-F 1 "Conn_01x04_Female" V 10850 3100 50  0000 L CNN
-F 2 "Connector_JST:JST_SH_SM04B-SRSS-TB_1x04-1MP_P1.00mm_Horizontal" H 10650 3500 50  0001 C CNN
-F 3 "~" H 10650 3500 50  0001 C CNN
-	1    10650 3500
+P 10350 3500
+F 0 "J8" H 10378 3476 50  0000 L CNN
+F 1 "Conn_01x04_Female" V 10550 3100 50  0000 L CNN
+F 2 "Connector_JST:JST_SH_SM04B-SRSS-TB_1x04-1MP_P1.00mm_Horizontal" H 10350 3500 50  0001 C CNN
+F 3 "~" H 10350 3500 50  0001 C CNN
+	1    10350 3500
 	1    0    0    -1
 $EndComp
@@
 L power:GND #PWR0125
 U 1 1 5F6942B2
-P 10450 3700
-F 0 "#PWR0125" H 10450 3450 50  0001 C CNN
-F 1 "GND" H 10455 3527 50  0000 C CNN
-F 2 "" H 10450 3700 50  0001 C CNN
-F 3 "" H 10450 3700 50  0001 C CNN
-	1    10450 3700
+P 10150 3700
+F 0 "#PWR0125" H 10150 3450 50  0001 C CNN
+F 1 "GND" H 10155 3527 50  0000 C CNN
+F 2 "" H 10150 3700 50  0001 C CNN
+F 3 "" H 10150 3700 50  0001 C CNN
+	1    10150 3700
 	1    0    0    -1
 $EndComp
@@
 L power:VCC #PWR0126
 U 1 1 5F6869FA
-P 10150 3600
-F 0 "#PWR0126" H 10150 3450 50  0001 C CNN
-F 1 "VCC" H 10167 3773 50  0000 C CNN
-F 2 "" H 10150 3600 50  0001 C CNN
-F 3 "" H 10150 3600 50  0001 C CNN
-	1    10150 3600
-	1    0    0    -1
-$EndComp
-Wire Wire Line
-	10450 3600 10150 3600
-Text GLabel 10450 3400 0    50   Input ~ 0
+P 9850 3600
+F 0 "#PWR0126" H 9850 3450 50  0001 C CNN
+F 1 "VCC" H 9867 3773 50  0000 C CNN
+F 2 "" H 9850 3600 50  0001 C CNN
+F 3 "" H 9850 3600 50  0001 C CNN
+	1    9850 3600
+	1    0    0    -1
+$EndComp
+Wire Wire Line
+	10150 3600 9850 3600
+Text GLabel 10150 3400 0    50   Input ~ 0
 A4
-Text GLabel 10450 3500 0    50   Input ~ 0
+Text GLabel 10150 3500 0    50   Input ~ 0
 A5
 $Comp
@@
 	1    0    0    -1
 $EndComp
+$Comp
+L Device:R R7
+U 1 1 5F7227DD
+P 10750 3600
+F 0 "R7" H 10820 3646 50  0000 L CNN
+F 1 "R" H 10820 3555 50  0000 L CNN
+F 2 "Resistor_THT:R_Axial_DIN0204_L3.6mm_D1.6mm_P2.54mm_Vertical" V 10680 3600 50  0001 C CNN
+F 3 "~" H 10750 3600 50  0001 C CNN
+	1    10750 3600
+	1    0    0    -1
+$EndComp
+$Comp
+L Device:R R8
+U 1 1 5F722F91
+P 10950 3600
+F 0 "R8" H 11020 3646 50  0000 L CNN
+F 1 "R" H 11020 3555 50  0000 L CNN
+F 2 "Resistor_THT:R_Axial_DIN0204_L3.6mm_D1.6mm_P2.54mm_Vertical" V 10880 3600 50  0001 C CNN
+F 3 "~" H 10950 3600 50  0001 C CNN
+	1    10950 3600
+	1    0    0    -1
+$EndComp
+Text GLabel 10750 3750 0    50   Input ~ 0
+A4
+Text GLabel 10950 3750 0    50   Input ~ 0
+A5
+$Comp
+L power:VCC #PWR0129
+U 1 1 5F7234B5
+P 10750 3450
+F 0 "#PWR0129" H 10750 3300 50  0001 C CNN
+F 1 "VCC" H 10767 3623 50  0000 C CNN
+F 2 "" H 10750 3450 50  0001 C CNN
+F 3 "" H 10750 3450 50  0001 C CNN
+	1    10750 3450
+	1    0    0    -1
+$EndComp
+$Comp
+L power:VCC #PWR0130
+U 1 1 5F723964
+P 10950 3450
+F 0 "#PWR0130" H 10950 3300 50  0001 C CNN
+F 1 "VCC" H 10967 3623 50  0000 C CNN
+F 2 "" H 10950 3450 50  0001 C CNN
+F 3 "" H 10950 3450 50  0001 C CNN
+	1    10950 3450
+	1    0    0    -1
+$EndComp
+$Comp
+L power:GND #PWR?
+U 1 1 5F749853
+P -1650 3000
+F 0 "#PWR?" H -1650 2750 50  0001 C CNN
+F 1 "GND" H -1645 2827 50  0000 C CNN
+F 2 "" H -1650 3000 50  0001 C CNN
+F 3 "" H -1650 3000 50  0001 C CNN
+	1    -1650 3000
+	1    0    0    -1
+$EndComp
+Wire Wire Line
+	-1500 2800 -1650 2800
+Wire Wire Line
+	-1500 2900 -2100 2900
+Wire Wire Line
+	-1650 3000 -1650 2800
+$Comp
+L power:VCC #PWR?
+U 1 1 5F748332
+P -2100 2900
+F 0 "#PWR?" H -2100 2750 50  0001 C CNN
+F 1 "VCC" H -2083 3073 50  0000 C CNN
+F 2 "" H -2100 2900 50  0001 C CNN
+F 3 "" H -2100 2900 50  0001 C CNN
+	1    -2100 2900
+	1    0    0    -1
+$EndComp
 Text GLabel -1500 2700 0    50   Input ~ 0
 VIN
-$Comp
-L power:GND #PWR0129
-U 1 1 5F6E2E0D
-P -1600 3100
-F 0 "#PWR0129" H -1600 2850 50  0001 C CNN
-F 1 "GND" H -1595 2927 50  0000 C CNN
-F 2 "" H -1600 3100 50  0001 C CNN
-F 3 "" H -1600 3100 50  0001 C CNN
-	1    -1600 3100
-	1    0    0    -1
-$EndComp
-$Comp
-L power:VCC #PWR0130
-U 1 1 5F6E4957
-P -1950 2900
-F 0 "#PWR0130" H -1950 2750 50  0001 C CNN
-F 1 "VCC" H -1933 3073 50  0000 C CNN
-F 2 "" H -1950 2900 50  0001 C CNN
-F 3 "" H -1950 2900 50  0001 C CNN
-	1    -1950 2900
-	1    0    0    -1
-$EndComp
-Wire Wire Line
-	-1500 2800 -1600 2800
-Wire Wire Line
-	-1500 2900 -1950 2900
-Wire Wire Line
-	-1600 2800 -1600 3100
 $EndSCHEMATC
