File: ver2/dippy.kicad_pcb (KiCad board)
At the start: 2 copper layers, 33.7 x 73.7 mm, 34 parts, among them J1 Screw_Terminal_01x02, J2 Screw_Terminal_01x03, J3 Screw_Terminal_01x04, J4 Conn_Coaxial, J5 Conn_02x03_Odd_Even, J6 Conn_01x04_Female, J7 Conn_01x03_Female, J8 Screw_Terminal_01x04, J9 Conn_01x03_Female, SW1 SW_Push_Dual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

Commit message: update
Parts:
- moved R5 5.47 mm to (137.4, 70.0), turned to 90 degrees
- moved R1 4.73 mm to (139.7, 65.0), turned to 270 degrees
- moved R7 2.79 mm to (140.5, 78.2)
- moved R4 2.47 mm to (140.5, 76.0)
- moved FTDI1 1.27 mm to (125.0, 60.7)
- moved R8 1.24 mm to (131.5, 73.7)
- moved J9 1.06 mm to (132.6, 66.1)
- moved C4 0.92 mm to (120.5, 74.1)
- moved U3 0.84 mm to (124.9, 74.9)
- moved C1 0.81 mm to (136.4, 75.8)
- moved C2 0.76 mm to (116.5, 74.1)
- moved AT1 0.53 mm to (137.2, 130.4)
- moved H3 0.46 mm to (144.9, 112.5)
- moved SW1 0.34 mm to (142.1, 72.3)
- moved J1 0.12 mm to (120.5, 67.1)
Routing:
- net VCC: track 69.9 -> 168.1 mm, vias 1 -> 3
- net GND: track 138.7 -> 231.7 mm, vias 7 -> 8
- net VIN: track 0.54 -> 46.9 mm
- net A5: track 0.00 -> 32.9 mm
- net RX0: track 7.04 -> 32.4 mm, vias 0 -> 2
- net TX0: track 13.7 -> 36.6 mm, vias 0 -> 2
- net A3: track 7.53 -> 29.7 mm, vias 0 -> 1
- net Net-(C1-Pad2): track 0.00 -> 17.0 mm, vias 0 -> 1
- net RST: track 56.4 -> 72.8 mm, vias 2 -> 1
- net A4: track 14.4 -> 27.7 mm, vias 1 -> 0
- net A0: track 7.86 -> 14.7 mm
- net Net-(C3-Pad1): track 0.00 -> 2.60 mm
- net Net-(AT1-Pad1): track 15.3 -> 15.1 mm, vias 0 -> 2
Other:
- board text added: "ver 2"
- board text removed: "RESET"
- board text removed: "qwiic"
- board text removed: "ver 1"

Commit message: update
Parts:
- added G***: LOGO, footprints:moth4, F.Cu at (143.4, 119.4)
Other:
- board text added: "1/GND"
- board text added: "2/MISO"
- board text added: "9/ANT"
- board text added: "ANT"
- board text removed: "1"
- board text removed: "9"
- board text removed: "AT"

Commit message: update
Parts:
- moved R7 0.15 mm to (140.4, 78.3)
- moved R4 0.15 mm to (140.4, 76.0)
Routing:
- net A4: track 27.7 -> 28.5 mm

Commit message: update
Routing:
- net GND: track 231.7 -> 233.2 mm

Commit message: update
Routing:
- net D5: track 14.5 -> 11.8 mm, vias 1 -> 0
Other:
- board text added: "VCC"
- board text removed: "D5"
Changed lines of the file:
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@@
   (general
     (thickness 1.6)
-    (drawings 79)
-    (tracks 498)
+    (drawings 81)
+    (tracks 496)
     (zones 0)
     (modules 35)
@@
     )
   )
+  (gr_text VCC (at 127.175 68.4) (layer F.SilkS)
+    (effects (font (size 0.85 0.85) (thickness 0.15)))
+  )
+  (gr_text GND (at 130.2 68.375) (layer F.SilkS)
+    (effects (font (size 0.85 0.85) (thickness 0.15)))
+  )
+  (gr_text VIN (at 133.025 68.375) (layer F.SilkS)
+    (effects (font (size 0.85 0.85) (thickness 0.15)))
+  )
   (gr_circle (center 137.1854 130.3274) (end 138.67892 131.2037) (layer F.SilkS) (width 0.12))
   (gr_text 2/MISO (at 121.67108 118.872) (layer F.SilkS)
@@
     (effects (font (size 0.85 0.85) (thickness 0.15)) (justify mirror))
   )
-  (gr_text DC-DC (at 130.2258 69.9516) (layer F.SilkS)
+  (gr_text DC-DC (at 130.10388 70.73646) (layer F.SilkS)
     (effects (font (size 1.2 1.2) (thickness 0.15)))
   )
@@
   (gr_text A2 (at 128.1176 87.0458 90) (layer B.SilkS)
     (effects (font (size 1 1) (thickness 0.16)) (justify mirror))
-  )
-  (gr_text D5 (at 130.1242 104.3686 90) (layer B.SilkS)
-    (effects (font (size 1 1) (thickness 0.15)) (justify mirror))
   )
   (gr_text RFM9x (at 125.8316 122.9868) (layer F.SilkS)
@@
   (segment (start 126.86137 84.455) (end 129.032 82.28437) (width 1) (layer B.Cu) (net 11))
   (segment (start 125.73 84.455) (end 126.86137 84.455) (width 1) (layer B.Cu) (net 11))
-  (segment (start 129.032 82.28437) (end 129.032 78.486) (width 1) (layer B.Cu) (net 11))
   (segment (start 135.12292 61.857281) (end 132.657241 64.32296) (width 1) (layer B.Cu) (net 11))
   (segment (start 135.12292 60.6552) (end 135.12292 61.857281) (width 1) (layer B.Cu) (net 11))
@@
   (segment (start 125.84684 64.40932) (end 125.84684 69.88048) (width 1) (layer B.Cu) (net 11))
   (segment (start 125.84684 69.88048) (end 125.9332 69.96684) (width 1) (layer B.Cu) (net 11))
-  (via (at 129.51968 77.91704) (size 0.8) (drill 0.4) (layers F.Cu B.Cu) (net 11))
-  (segment (start 129.032 78.486) (end 129.032 78.40472) (width 1) (layer B.Cu) (net 11))
-  (segment (start 129.032 78.40472) (end 129.51968 77.91704) (width 1) (layer B.Cu) (net 11))
-  (segment (start 129.51968 77.91704) (end 130.07848 77.35824) (width 1) (layer F.Cu) (net 11))
-  (segment (start 130.07848 77.35824) (end 130.07848 73.46696) (width 1) (layer F.Cu) (net 11))
   (segment (start 130.07848 73.46696) (end 128.03632 71.4248) (width 1) (layer F.Cu) (net 11))
   (segment (start 128.03632 71.4248) (end 126.746 71.4248) (width 1) (layer F.Cu) (net 11))
   (segment (start 125.9332 70.612) (end 125.9332 69.96684) (width 1) (layer F.Cu) (net 11))
   (segment (start 126.746 71.4248) (end 125.9332 70.612) (width 1) (layer F.Cu) (net 11))
+  (segment (start 129.032 82.28437) (end 129.032 82.268) (width 1) (layer B.Cu) (net 11))
+  (segment (start 129.032 82.268) (end 129.4 81.9) (width 1) (layer B.Cu) (net 11))
+  (segment (start 129.4 81.9) (end 129.4 75.95) (width 1) (layer B.Cu) (net 11))
+  (via (at 130.25 75.1) (size 0.8) (drill 0.4) (layers F.Cu B.Cu) (net 11))
+  (segment (start 129.4 75.95) (end 130.25 75.1) (width 1) (layer B.Cu) (net 11))
+  (segment (start 130.07848 74.92848) (end 130.07848 73.46696) (width 1) (layer F.Cu) (net 11))
+  (segment (start 130.25 75.1) (end 130.07848 74.92848) (width 1) (layer F.Cu) (net 11))
   (segment (start 127.508 81.26837) (end 126.86137 81.915) (width 1) (layer B.Cu) (net 12))
   (segment (start 126.86137 81.915) (end 125.73 81.915) (width 1) (layer B.Cu) (net 12) (status 20))
@@
   (segment (start 145.57248 75.97648) (end 145.59788 75.95108) (width 1) (layer B.Cu) (net 22))
   (segment (start 145.4531 75.97648) (end 145.57248 75.97648) (width 1) (layer B.Cu) (net 22))
-  (via (at 128.3208 104.3178) (size 1.78) (drill 0.89) (layers F.Cu B.Cu) (net 23))
-  (segment (start 125.73 104.775) (end 127.8636 104.775) (width 1) (layer F.Cu) (net 23))
-  (segment (start 127.8636 104.775) (end 128.3208 104.3178) (width 1) (layer F.Cu) (net 23))
   (segment (start 125.73 104.775) (end 120.4722 104.775) (width 1) (layer B.Cu) (net 23))
   (segment (start 116.5352 108.2548) (end 118.9228 108.2548) (width 1) (layer B.Cu) (net 23))
