File: ver2/dippy.sch (KiCad schematic (older format))
At the start: 34 parts, among them J1 Screw_Terminal_01x02, J2 Screw_Terminal_01x03, J3 Screw_Terminal_01x04, J4 Conn_Coaxial, J5 Conn_02x03_Odd_Even, J6 Conn_01x04_Female, J7 Conn_01x03_Female, J8 Screw_Terminal_01x04, J9 Conn_01x03_Female, SW1 SW_Push_Dual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

Commit message: update
Other:
- moved on the sheet: R2
Changed lines of the file:
@@
 L Device:R R2
 U 1 1 5F322886
-P 7750 5600
-F 0 "R2" H 7820 5646 50  0000 L CNN
-F 1 "10K" H 7820 5555 50  0000 L CNN
-F 2 "Resistor_THT:R_Axial_DIN0204_L3.6mm_D1.6mm_P5.08mm_Horizontal" V 7680 5600 50  0001 C CNN
-F 3 "~" H 7750 5600 50  0001 C CNN
-	1    7750 5600
+P 8400 5550
+F 0 "R2" H 8470 5596 50  0000 L CNN
+F 1 "10K" H 8470 5505 50  0000 L CNN
+F 2 "Resistor_THT:R_Axial_DIN0204_L3.6mm_D1.6mm_P5.08mm_Horizontal" V 8330 5550 50  0001 C CNN
+F 3 "~" H 8400 5550 50  0001 C CNN
+	1    8400 5550
 	1    0    0    -1
 $EndComp
@@
 L power:VCC #PWR0113
 U 1 1 5F322DF7
-P 7750 5450
-F 0 "#PWR0113" H 7750 5300 50  0001 C CNN
-F 1 "VCC" H 7767 5623 50  0000 C CNN
-F 2 "" H 7750 5450 50  0001 C CNN
-F 3 "" H 7750 5450 50  0001 C CNN
-	1    7750 5450
+P 8400 5400
+F 0 "#PWR0113" H 8400 5250 50  0001 C CNN
+F 1 "VCC" H 8417 5573 50  0000 C CNN
+F 2 "" H 8400 5400 50  0001 C CNN
+F 3 "" H 8400 5400 50  0001 C CNN
+	1    8400 5400
 	1    0    0    -1
 $EndComp
@@
 Wire Wire Line
 	9250 3550 8900 3550
-Text GLabel 7750 5750 0    50   Input ~ 0
+Text GLabel 8400 5700 0    50   Input ~ 0
 A0
 Text GLabel 6350 4350 0    50   Input ~ 0

Commit message: update
Other:
- note added: "DC-DC"
- note added: "LDO"
- moved on the sheet: C2, C4, C5, J1, J9, U3
Changed lines of the file:
@@
 $EndComp
 Wire Wire Line
-	3050 5450 2700 5450
-Wire Wire Line
-	2250 5550 2250 5750
+	3950 5400 3600 5400
+Wire Wire Line
+	3150 5500 3150 5700
 $Comp
 L Device:C C2
 U 1 1 5F27AAEF
-P 2700 5600
-F 0 "C2" H 2815 5646 50  0000 L CNN
-F 1 "0.1u" H 2815 5555 50  0000 L CNN
-F 2 "Capacitor_THT:C_Disc_D3.0mm_W1.6mm_P2.50mm" H 2738 5450 50  0001 C CNN
-F 3 "~" H 2700 5600 50  0001 C CNN
-	1    2700 5600
-	1    0    0    -1
-$EndComp
-Connection ~ 2700 5450
-Wire Wire Line
-	2700 5450 2250 5450
-Wire Wire Line
-	3350 5750 2700 5750
-Wire Wire Line
-	2700 5750 2250 5750
-Connection ~ 2700 5750
+P 3600 5550
+F 0 "C2" H 3715 5596 50  0000 L CNN
+F 1 "0.1u" H 3715 5505 50  0000 L CNN
+F 2 "Capacitor_THT:C_Disc_D3.0mm_W1.6mm_P2.50mm" H 3638 5400 50  0001 C CNN
+F 3 "~" H 3600 5550 50  0001 C CNN
+	1    3600 5550
+	1    0    0    -1
+$EndComp
+Connection ~ 3600 5400
+Wire Wire Line
+	3600 5400 3150 5400
+Wire Wire Line
+	4250 5700 3600 5700
+Wire Wire Line
+	3600 5700 3150 5700
+Connection ~ 3600 5700
 $Comp
 L power:GND #PWR0104
 U 1 1 5F27BAB1
-P 3350 5900
-F 0 "#PWR0104" H 3350 5650 50  0001 C CNN
-F 1 "GND" H 3355 5727 50  0000 C CNN
-F 2 "" H 3350 5900 50  0001 C CNN
-F 3 "" H 3350 5900 50  0001 C CNN
-	1    3350 5900
-	1    0    0    -1
-$EndComp
-Connection ~ 3350 5750
-Wire Wire Line
-	3650 5450 3800 5450
+P 4250 5850
+F 0 "#PWR0104" H 4250 5600 50  0001 C CNN
+F 1 "GND" H 4255 5677 50  0000 C CNN
+F 2 "" H 4250 5850 50  0001 C CNN
+F 3 "" H 4250 5850 50  0001 C CNN
+	1    4250 5850
+	1    0    0    -1
+$EndComp
+Connection ~ 4250 5700
+Wire Wire Line
+	4550 5400 4700 5400
 $Comp
 L Device:C C4
 U 1 1 5F27C5A9
-P 3800 5600
-F 0 "C4" H 3915 5646 50  0000 L CNN
-F 1 "0.1u" H 3915 5555 50  0000 L CNN
-F 2 "Capacitor_THT:C_Disc_D3.0mm_W1.6mm_P2.50mm" H 3838 5450 50  0001 C CNN
-F 3 "~" H 3800 5600 50  0001 C CNN
-	1    3800 5600
-	1    0    0    -1
-$EndComp
-Connection ~ 3800 5450
-Wire Wire Line
-	3800 5450 4250 5450
-Connection ~ 4250 5450
-Wire Wire Line
-	4250 5450 4400 5450
-Wire Wire Line
-	3350 5750 3350 5900
-Wire Wire Line
-	3350 5750 3800 5750
-Wire Wire Line
-	3800 5750 4250 5750
-Connection ~ 3800 5750
+P 4700 5550
+F 0 "C4" H 4815 5596 50  0000 L CNN
+F 1 "0.1u" H 4815 5505 50  0000 L CNN
+F 2 "Capacitor_THT:C_Disc_D3.0mm_W1.6mm_P2.50mm" H 4738 5400 50  0001 C CNN
+F 3 "~" H 4700 5550 50  0001 C CNN
+	1    4700 5550
+	1    0    0    -1
+$EndComp
+Connection ~ 4700 5400
+Wire Wire Line
+	4700 5400 5150 5400
+Connection ~ 5150 5400
+Wire Wire Line
+	5150 5400 5300 5400
+Wire Wire Line
+	4250 5700 4250 5850
+Wire Wire Line
+	4250 5700 4700 5700
+Wire Wire Line
+	4700 5700 5150 5700
+Connection ~ 4700 5700
 $Comp
 L RF_Module:RFM95W-915S2 U2
@@
 	-1   0    0    1
 $EndComp
-Text GLabel 2700 4950 0    50   Input ~ 0
+Text GLabel 3600 4900 0    50   Input ~ 0
 VIN
 Wire Wire Line
-	2700 4950 2700 5450
+	3600 4900 3600 5400
 Text GLabel 7500 2450 2    50   Input ~ 0
 D6
@@
 L power:VCC #PWR0105
 U 1 1 5F27EDB1
-P 4400 5450
-F 0 "#PWR0105" H 4400 5300 50  0001 C CNN
-F 1 "VCC" H 4417 5623 50  0000 C CNN
-F 2 "" H 4400 5450 50  0001 C CNN
-F 3 "" H 4400 5450 50  0001 C CNN
-	1    4400 5450
+P 5300 5400
+F 0 "#PWR0105" H 5300 5250 50  0001 C CNN
+F 1 "VCC" H 5317 5573 50  0000 C CNN
+F 2 "" H 5300 5400 50  0001 C CNN
+F 3 "" H 5300 5400 50  0001 C CNN
+	1    5300 5400
 	1    0    0    -1
 $EndComp
@@
 L Device:C C5
 U 1 1 5F27CEC8
-P 4250 5600
-F 0 "C5" H 4365 5646 50  0000 L CNN
-F 1 "10u" H 4365 5555 50  0000 L CNN
-F 2 "Capacitor_THT:CP_Radial_D5.0mm_P2.50mm" H 4288 5450 50  0001 C CNN
-F 3 "~" H 4250 5600 50  0001 C CNN
-	1    4250 5600
+P 5150 5550
+F 0 "C5" H 5265 5596 50  0000 L CNN
+F 1 "10u" H 5265 5505 50  0000 L CNN
+F 2 "Capacitor_THT:CP_Radial_D5.0mm_P2.50mm" H 5188 5400 50  0001 C CNN
+F 3 "~" H 5150 5550 50  0001 C CNN
+	1    5150 5550
 	1    0    0    -1
 $EndComp
@@
 L Regulator_Linear:MCP1700-3302E_TO92 U3
 U 1 1 5F67A451
-P 3350 5450
-F 0 "U3" H 3350 5208 50  0000 C CNN
-F 1 "MCP1700-3302E_TO92" H 3350 5299 50  0000 C CNN
-F 2 "Package_TO_SOT_THT:TO-92_Inline" H 3350 5250 50  0001 C CIN
-F 3 "http://ww1.microchip.com/downloads/en/DeviceDoc/20001826D.pdf" H 3350 5450 50  0001 C CNN
-	1    3350 5450
+P 4250 5400
+F 0 "U3" H 4250 5158 50  0000 C CNN
+F 1 "MCP1700-3302E_TO92" H 4250 5249 50  0000 C CNN
+F 2 "Package_TO_SOT_THT:TO-92_Inline" H 4250 5200 50  0001 C CIN
+F 3 "http://ww1.microchip.com/downloads/en/DeviceDoc/20001826D.pdf" H 4250 5400 50  0001 C CNN
+	1    4250 5400
 	1    0    0    1
 $EndComp
@@
 L Connector:Conn_01x03_Female J9
 U 1 1 5F6DC6E3
-P -1300 2800
-F 0 "J9" H -1272 2826 50  0000 L CNN
-F 1 "Conn_01x03_Female" H -1272 2735 50  0000 L CNN
-F 2 "Connector_PinSocket_2.54mm:PinSocket_1x03_P2.54mm_Vertical" H -1300 2800 50  0001 C CNN
-F 3 "~" H -1300 2800 50  0001 C CNN
-	1    -1300 2800
+P 1850 5450
+F 0 "J9" H 1878 5476 50  0000 L CNN
+F 1 "Conn_01x03_Female" V 2050 5050 50  0000 L CNN
+F 2 "Connector_PinSocket_2.54mm:PinSocket_1x03_P2.54mm_Vertical" H 1850 5450 50  0001 C CNN
+F 3 "~" H 1850 5450 50  0001 C CNN
+	1    1850 5450
 	1    0    0    -1
 $EndComp
@@
 L power:GND #PWR0125
 U 1 1 5F749853
-P -1650 3000
-F 0 "#PWR0125" H -1650 2750 50  0001 C CNN
-F 1 "GND" H -1645 2827 50  0000 C CNN
-F 2 "" H -1650 3000 50  0001 C CNN
-F 3 "" H -1650 3000 50  0001 C CNN
-	1    -1650 3000
-	1    0    0    -1
-$EndComp
-Wire Wire Line
-	-1500 2800 -1650 2800
-Wire Wire Line
-	-1500 2900 -2100 2900
-Wire Wire Line
-	-1650 3000 -1650 2800
+P 1500 5650
+F 0 "#PWR0125" H 1500 5400 50  0001 C CNN
+F 1 "GND" H 1505 5477 50  0000 C CNN
+F 2 "" H 1500 5650 50  0001 C CNN
+F 3 "" H 1500 5650 50  0001 C CNN
+	1    1500 5650
+	1    0    0    -1
+$EndComp
+Wire Wire Line
+	1650 5450 1500 5450
+Wire Wire Line
+	1650 5550 1050 5550
+Wire Wire Line
+	1500 5650 1500 5450
 $Comp
 L power:VCC #PWR0126
 U 1 1 5F748332
-P -2100 2900
-F 0 "#PWR0126" H -2100 2750 50  0001 C CNN
-F 1 "VCC" H -2083 3073 50  0000 C CNN
-F 2 "" H -2100 2900 50  0001 C CNN
-F 3 "" H -2100 2900 50  0001 C CNN
-	1    -2100 2900
-	1    0    0    -1
-$EndComp
-Text GLabel -1500 2700 0    50   Input ~ 0
+P 1050 5550
+F 0 "#PWR0126" H 1050 5400 50  0001 C CNN
+F 1 "VCC" H 1067 5723 50  0000 C CNN
+F 2 "" H 1050 5550 50  0001 C CNN
+F 3 "" H 1050 5550 50  0001 C CNN
+	1    1050 5550
+	1    0    0    -1
+$EndComp
+Text GLabel 1650 5350 0    50   Input ~ 0
 VIN
 $Comp
@@
 L Connector:Screw_Terminal_01x02 J1
 U 1 1 5F6EF08A
-P 2050 5550
-F 0 "J1" H 1968 5225 50  0000 C CNN
-F 1 "Screw_Terminal_01x02" H 1968 5316 50  0000 C CNN
-F 2 "TerminalBlock_Phoenix:TerminalBlock_Phoenix_PT-1,5-2-3.5-H_1x02_P3.50mm_Horizontal" H 2050 5550 50  0001 C CNN
-F 3 "~" H 2050 5550 50  0001 C CNN
-	1    2050 5550
+P 2950 5500
+F 0 "J1" H 2868 5175 50  0000 C CNN
+F 1 "Screw_Terminal_01x02" H 2868 5266 50  0000 C CNN
+F 2 "TerminalBlock_Phoenix:TerminalBlock_Phoenix_PT-1,5-2-3.5-H_1x02_P3.50mm_Horizontal" H 2950 5500 50  0001 C CNN
+F 3 "~" H 2950 5500 50  0001 C CNN
+	1    2950 5500
 	-1   0    0    1
 $EndComp
+Text Notes 1200 5150 0    118  ~ 0
+DC-DC
+Text Notes 4000 5000 0    118  ~ 0
+LDO
 $EndSCHEMATC

Commit message: update
Other:
- moved on the sheet: D1, R6, SW1
Changed lines of the file:
@@
 A0
-Wire Wire Line
-	1150 1600 1150 1700
-Connection ~ 1150 1700
-Wire Wire Line
-	1150 1700 1150 1850
 Wire Wire Line
 	2500 3050 2500 3150
@@
 L Device:LED D1
 U 1 1 5F57E191
-P 4950 1600
-F 0 "D1" V 4989 1482 50  0000 R CNN
-F 1 "LED" V 4898 1482 50  0000 R CNN
-F 2 "LED_THT:LED_D3.0mm" H 4950 1600 50  0001 C CNN
-F 3 "~" H 4950 1600 50  0001 C CNN
-	1    4950 1600
+P 1850 2150
+F 0 "D1" V 1889 2032 50  0000 R CNN
+F 1 "LED" V 1798 2032 50  0000 R CNN
+F 2 "LED_THT:LED_D3.0mm" H 1850 2150 50  0001 C CNN
+F 3 "~" H 1850 2150 50  0001 C CNN
+	1    1850 2150
 	0    -1   -1   0
 $EndComp
-Text GLabel 4950 1450 0    50   Input ~ 0
+Text GLabel 1850 2000 0    50   Input ~ 0
 D5
 $Comp
 L power:GND #PWR0124
 U 1 1 5F5807E4
-P 4950 2050
-F 0 "#PWR0124" H 4950 1800 50  0001 C CNN
-F 1 "GND" H 4955 1877 50  0000 C CNN
-F 2 "" H 4950 2050 50  0001 C CNN
-F 3 "" H 4950 2050 50  0001 C CNN
-	1    4950 2050
+P 1850 2600
+F 0 "#PWR0124" H 1850 2350 50  0001 C CNN
+F 1 "GND" H 1855 2427 50  0000 C CNN
+F 2 "" H 1850 2600 50  0001 C CNN
+F 3 "" H 1850 2600 50  0001 C CNN
+	1    1850 2600
 	1    0    0    -1
 $EndComp
@@
 L Device:R R6
 U 1 1 5F59A5EA
-P 4950 1900
-F 0 "R6" H 5020 1946 50  0000 L CNN
-F 1 "300R" H 5020 1855 50  0000 L CNN
-F 2 "Resistor_THT:R_Axial_DIN0204_L3.6mm_D1.6mm_P5.08mm_Horizontal" V 4880 1900 50  0001 C CNN
-F 3 "~" H 4950 1900 50  0001 C CNN
-	1    4950 1900
+P 1850 2450
+F 0 "R6" H 1920 2496 50  0000 L CNN
+F 1 "300R" H 1920 2405 50  0000 L CNN
+F 2 "Resistor_THT:R_Axial_DIN0204_L3.6mm_D1.6mm_P5.08mm_Horizontal" V 1780 2450 50  0001 C CNN
+F 3 "~" H 1850 2450 50  0001 C CNN
+	1    1850 2450
 	1    0    0    -1
 $EndComp
 Text GLabel 2650 1700 1    50   Input ~ 0
 RST
-Wire Wire Line
-	1150 1700 2850 1700
 Text GLabel 9650 5650 3    50   Input ~ 0
 RST
@@
 L Switch:SW_Push_Dual SW1
 U 1 1 5F6B37D1
-P -1200 1050
-F 0 "SW1" H -1200 1335 50  0000 C CNN
-F 1 "SW_Push_Dual" H -1200 1244 50  0000 C CNN
-F 2 "Button_Switch_THT:SW_TH_Tactile_Omron_B3F-10xx" H -1200 1250 50  0001 C CNN
-F 3 "~" H -1200 1250 50  0001 C CNN
-	1    -1200 1050
-	1    0    0    -1
-$EndComp
-Text GLabel -1400 1050 0    50   Input ~ 0
+P 4950 1700
+F 0 "SW1" H 4950 1985 50  0000 C CNN
+F 1 "SW_Push_Dual" H 4950 1894 50  0000 C CNN
+F 2 "Button_Switch_THT:SW_TH_Tactile_Omron_B3F-10xx" H 4950 1900 50  0001 C CNN
+F 3 "~" H 4950 1900 50  0001 C CNN
+	1    4950 1700
+	1    0    0    -1
+$EndComp
+Text GLabel 4750 1700 0    50   Input ~ 0
 RST
 Wire Wire Line
-	-1400 1050 -1400 1250
-Wire Wire Line
-	-1000 1050 -1000 1250
+	4750 1700 4750 1900
+Wire Wire Line
+	5150 1700 5150 1900
 $Comp
 L power:GND #PWR0128
 U 1 1 5F6BD020
-P -1000 1250
-F 0 "#PWR0128" H -1000 1000 50  0001 C CNN
-F 1 "GND" H -995 1077 50  0000 C CNN
-F 2 "" H -1000 1250 50  0001 C CNN
-F 3 "" H -1000 1250 50  0001 C CNN
-	1    -1000 1250
-	1    0    0    -1
-$EndComp
-Connection ~ -1000 1250
+P 5150 1900
+F 0 "#PWR0128" H 5150 1650 50  0001 C CNN
+F 1 "GND" H 5155 1727 50  0000 C CNN
+F 2 "" H 5150 1900 50  0001 C CNN
+F 3 "" H 5150 1900 50  0001 C CNN
+	1    5150 1900
+	1    0    0    -1
+$EndComp
+Connection ~ 5150 1900
 $Comp
 L Connector:Conn_01x03_Female J9
@@
 Text Notes 4000 5000 0    118  ~ 0
 LDO
+Wire Wire Line
+	1150 1700 1150 1850
+Wire Wire Line
+	1150 1600 1150 1700
+Connection ~ 1150 1700
+Wire Wire Line
+	1150 1700 2850 1700
 $EndSCHEMATC

Commit message: update
Other:
- note added: "4) Battery Level"
- note removed: "4) Voltage\nMeausurement"
Changed lines of the file:
@@
 	5500 3950 800  3950
 Text Notes 9100 1050 0    118  ~ 0
-4) Voltage\nMeausurement
+4) Battery Level
 Wire Notes Line
 	11050 2600 8750 2600
