File: old/ver3_X/dippy.kicad_pcb (KiCad board)
At the start: 2 copper layers, 46.6 x 79.2 mm, 38 parts, among them J1 Screw_Terminal_01x02, J10 Conn_01x05_Female, J2 Screw_Terminal_01x03, J3 Screw_Terminal_01x05, J4 Conn_Coaxial, J5 Conn_02x03_Odd_Even, J6 Conn_01x04_Female, J7 Conn_01x05_Female, J8 Screw_Terminal_01x04, J9 Conn_01x03_Female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

Commit message: update
Parts:
- removed R9: 10K, Resistor_THT:R_Axial_DIN0204_L3.6mm_D1.6mm_P7.62mm_Horizontal
- added J11: Conn_01x03_Female, Connector_PinSocket_2.54mm:PinSocket_1x03_P2.54mm_Vertical, F.Cu at (-100.0, 52.5)
- J7: value Conn_01x05_Female -> Conn_01x03_Female; footprint Connector_PinSocket_2.54mm:PinSocket_1x05_P2.54mm_Vertical -> Connector_PinSocket_2.54mm:PinSocket_1x03_P2.54mm_Vertical; moved to B.Cu
- moved J7 19.7 mm to (-108.2, 27.4), turned to 180 degrees
- moved G*** 13.7 mm to (-88.5, 62.5), turned to 20 degrees
- moved C3 8.44 mm to (-102.3, 40.0), turned to 90 degrees
- moved C6 6.28 mm to (-99.5, 35.0), turned to 270 degrees
- moved R2 5.81 mm to (-96.8, 37.7), turned to 0 degrees
- moved J6 1.98 mm to (-100.0, 19.4)
- moved R8 1.36 mm to (-110.0, 13.7)
- moved C1 1.31 mm to (-94.2, -2.03)
- moved C2 1.30 mm to (-122.0, 13.6)
- moved C4 1.30 mm to (-122.0, 16.7)
- moved C5 1.01 mm to (-116.9, 36.6)
- moved R7 0.58 mm to (-97.0, 10.9)
- moved J9 0.43 mm to (-109.5, 4.35)
- moved J10 0.35 mm to (-117.9, 22.1)
- renumbered FTDI to FTDI1
Connections:
- J2 pad 3: A2 -> A0
- J7 pad 3: A0 -> GND
- R2 pad 2: A2 -> A0
Routing:
- net A2: track 32.5 -> 3.14 mm
- net D3: track 37.1 -> 15.8 mm, vias 1 -> 0
- net A1: track 24.0 -> 3.14 mm
- net GND: track 336.4 -> 349.3 mm
- net A0: track 23.5 -> 35.7 mm
- net Net-(C3-Pad1): track 12.1 -> 4.73 mm
- net A3: track 112.2 -> 105.9 mm, vias 0 -> 1
- net VCC: track 185.3 -> 180.7 mm
- net VIN: track 56.7 -> 53.4 mm
- net A5: track 24.2 -> 21.3 mm
- net SCK: track 50.4 -> 47.7 mm, vias 2 -> 3
- net RST: track 115.1 -> 112.5 mm
- net A4: track 38.1 -> 36.5 mm
- net Net-(C1-Pad2): track 4.13 -> 3.34 mm
- net TX0: track 34.8 -> 35.5 mm
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Other:
- board text added: "A4"
- board text added: "A5"
- board text added: "pvos.org/ mothbot"
- board text added: "ver3"
- board text removed: "A1"
- board text removed: "A2"
- board text removed: "A4/"
- board text removed: "A5/"
- board text removed: "MOTHBOT"
- board text removed: "http://pvos.org/"
- board text removed: "ver:3"
