File: ver4/dippy.kicad_pcb (KiCad board)
At the start: 2 copper layers, 46.6 x 79.2 mm, 40 parts, among them J1 Screw_Terminal_01x02, J10 Conn_01x06_Female, J11 Conn_01x04_Female, J12 Conn_01x02_Female, J2 Screw_Terminal_01x03, J3 Screw_Terminal_01x06, J4 Conn_Coaxial, J5 Conn_02x03_Odd_Even, J6 Conn_01x04_Female, J7 Conn_01x05_Female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

Commit message: update
Parts:
- moved G*** 2.79 mm to (-114.1, 7.32), turned to 30 degrees
- moved J3 0.11 mm to (-91.1, 49.8)
Other:
- board text added: "(U1 'top')"
- board text added: "M2.5"
- board text added: "v4"
- board text removed: "(M2.5)"
- board text removed: "VER:3"

Commit message: update
Parts:
- moved C4 0.83 mm to (-92.5, 55.1)
- moved C2 0.38 mm to (-92.5, 57.7)
- renumbered AT1 to ANT1
Routing:
- net GND: track 338.5 -> 340.8 mm
- net VCC: track 212.4 -> 213.3 mm
Other:
- board text added: "ANT"
- board text removed: "AT1"
Changed lines of the file:
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@@
     (thickness 1.6)
     (drawings 88)
-    (tracks 630)
+    (tracks 638)
     (zones 0)
     (modules 40)
@@
   )
   (module Capacitor_THT:C_Disc_D4.3mm_W1.9mm_P5.00mm (layer F.Cu)
-    (at -92.569 54.286)
+    (at -92.45 55.11)
     (descr "C, Disc series, Radial, pin pitch=5.00mm, , diameter*width=4.3*1.9mm^2, Capacitor, http://www.vishay.com/docs/45233/krseries.pdf")
     (tags "C Disc series Radial pin pitch 5.00mm  diameter 4.3mm width 1.9mm Capacitor")
@@
   )
   (module Capacitor_THT:C_Disc_D4.3mm_W1.9mm_P5.00mm (layer F.Cu)
-    (at -92.569 57.334)
+    (at -92.45 57.7)
     (descr "C, Disc series, Radial, pin pitch=5.00mm, , diameter*width=4.3*1.9mm^2, Capacitor, http://www.vishay.com/docs/45233/krseries.pdf")
     (tags "C Disc series Radial pin pitch 5.00mm  diameter 4.3mm width 1.9mm Capacitor")
@@
   (module footprints:RFM95 (layer F.Cu)
     (at -95.026 13.575 180)
-    (fp_text reference U2 (at 1.799 -1.7 180) (layer F.SilkS)
+    (fp_text reference U2 (at -1.866 12.895 270) (layer F.SilkS)
       (effects (font (size 1 1) (thickness 0.15)))
     )
@@
     (descr "CP, Radial series, Radial, pin pitch=2.50mm, , diameter=5mm, Electrolytic Capacitor")
     (tags "CP Radial series Radial pin pitch 2.50mm  diameter 5mm Electrolytic Capacitor")
-    (fp_text reference C5 (at 4.375 -1.975 180) (layer F.SilkS)
+    (fp_text reference C5 (at -1.565 2.365 180) (layer F.SilkS)
       (effects (font (size 1 1) (thickness 0.15)))
     )
@@
     (descr "Through hole straight socket strip, 1x01, 2.54mm pitch, single row (from Kicad 4.0.7), script generated")
     (tags "Through hole socket strip THT 1x01 2.54mm single row")
-    (fp_text reference AT1 (at 0.166 -2.658) (layer F.SilkS)
+    (fp_text reference ANT1 (at -0.154 -2.643) (layer F.SilkS)
       (effects (font (size 1 1) (thickness 0.15)))
     )
@@
     (effects (font (size 0.85 0.85) (thickness 0.15)) (justify mirror))
   )
-  (gr_text AT1 (at -120.6 4.95 270) (layer F.SilkS)
+  (gr_text ANT (at -120.64 4.73 90) (layer F.SilkS)
     (effects (font (size 0.85 0.85) (thickness 0.15)))
   )
-  (gr_text GND (at -123.6 4.525 270) (layer F.SilkS)
+  (gr_text GND (at -123.56 4.32 90) (layer F.SilkS)
     (effects (font (size 0.85 0.85) (thickness 0.15)))
   )
-  (gr_text GND (at -117.75 4.525 270) (layer F.SilkS)
+  (gr_text GND (at -117.93 4.35 90) (layer F.SilkS)
     (effects (font (size 0.85 0.85) (thickness 0.15)))
   )
@@
   (segment (start -128.600009 17.744991) (end -127.03 19.315) (width 1) (layer F.Cu) (net 4))
   (segment (start -110.301 64.876) (end -110.301 67.422) (width 1) (layer F.Cu) (net 4))
-  (segment (start -88.422 57.712) (end -88.044 57.334) (width 1) (layer F.Cu) (net 4))
-  (segment (start -88.422 64.375) (end -88.422 57.712) (width 1) (layer F.Cu) (net 4))
   (segment (start -104.805 75.805) (end -102.425 73.425) (width 1) (layer F.Cu) (net 4))
   (segment (start -126.125 70.946) (end -126.125 74.270002) (width 1) (layer F.Cu) (net 4))
@@
   (segment (start -104.135 65.335) (end -103.825 65.025) (width 1) (layer B.Cu) (net 4))
   (segment (start -104.135 70.265) (end -104.135 65.335) (width 1) (layer B.Cu) (net 4))
-  (segment (start -87.569 57.334) (end -87.569 54.286) (width 1) (layer F.Cu) (net 4))
   (segment (start -88.175 53.68) (end -87.569 54.286) (width 1) (layer F.Cu) (net 4))
   (segment (start -88.175 46.5) (end -88.175 53.68) (width 1) (layer F.Cu) (net 4))
@@
   (segment (start -124.6 53.29) (end -124.6 55.06) (width 1) (layer B.Cu) (net 4))
   (segment (start -123.63 52.32) (end -124.6 53.29) (width 1) (layer B.Cu) (net 4))
+  (segment (start -87.459 63.412) (end -88.422 64.375) (width 1) (layer F.Cu) (net 4))
+  (segment (start -87.459 57.984) (end -87.459 63.412) (width 1) (layer F.Cu) (net 4))
+  (segment (start -87.45 55.11) (end -87.518 55.11) (width 1) (layer F.Cu) (net 4))
+  (segment (start -87.518 55.11) (end -87.569 55.059) (width 1) (layer F.Cu) (net 4))
+  (segment (start -87.569 57.334) (end -87.569 55.059) (width 1) (layer F.Cu) (net 4))
+  (segment (start -87.569 55.059) (end -87.569 54.286) (width 1) (layer F.Cu) (net 4))
+  (segment (start -87.45 57.7) (end -87.45 55.11) (width 1) (layer F.Cu) (net 4))
   (segment (start -107.686 73.244) (end -107.505 73.425) (width 1) (layer F.Cu) (net 5))
   (segment (start -107.761 73.169) (end -107.505 73.425) (width 1) (layer F.Cu) (net 5))
   (segment (start -99.125 48.675) (end -99.45 48.35) (width 1) (layer F.Cu) (net 5))
   (segment (start -98.425 48.675) (end -99.125 48.675) (width 1) (layer F.Cu) (net 5))
-  (segment (start -98.425 48.675) (end -92.85 48.675) (width 1) (layer F.Cu) (net 5))
   (segment (start -99.325 48.675) (end -98.425 48.675) (width 1) (layer F.Cu) (net 5))
   (segment (start -107.647 67.897) (end -107.761 68.011) (width 1) (layer F.Cu) (net 5))
   (segment (start -107.286 67.897) (end -107.647 67.897) (width 1) (layer F.Cu) (net 5))
   (segment (start -90.975 49.825) (end -91.65 49.15) (width 1) (layer F.Cu) (net 5))
-  (segment (start -92.475 57.428) (end -92.569 57.334) (width 1) (layer F.Cu) (net 5))
   (segment (start -99.575 51.52) (end -97.335 53.76) (width 1) (layer F.Cu) (net 5))
   (segment (start -99.575 48.7) (end -99.575 51.52) (width 1) (layer F.Cu) (net 5))
   (segment (start -107.505 73.425) (end -107.286 73.206) (width 1) (layer F.Cu) (net 5))
-  (segment (start -90.425 51.025) (end -91.6 49.85) (width 1) (layer F.Cu) (net 5))
-  (segment (start -92.569 57.334) (end -90.425 55.19) (width 1) (layer F.Cu) (net 5))
-  (segment (start -90.425 55.19) (end -90.425 51.025) (width 1) (layer F.Cu) (net 5))
-  (segment (start -91.675 49.85) (end -92.85 48.675) (width 1) (layer F.Cu) (net 5))
-  (segment (start -91.6 49.85) (end -91.675 49.85) (width 1) (layer F.Cu) (net 5))
   (segment (start -98.709 62.25) (end -99.227 61.732) (width 1) (layer F.Cu) (net 5))
   (segment (start -99.227 61.732) (end -99.227 62.877) (width 1) (layer F.Cu) (net 5))
@@
   (segment (start -96.106 73.689) (end -96.266 73.529) (width 1) (layer F.Cu) (net 5))
   (segment (start -96.106 73.719) (end -96.106 73.689) (width 1) (layer F.Cu) (net 5))
-  (segment (start -92.569 62.511) (end -92.19 62.89) (width 1) (layer B.Cu) (net 5))
-  (segment (start -92.569 57.334) (end -92.569 62.511) (width 1) (layer B.Cu) (net 5))
+  (segment (start -90.425 55.95) (end -92.459 57.984) (width 1) (layer F.Cu) (net 5))
+  (segment (start -90.425 51.025) (end -90.425 55.95) (width 1) (layer F.Cu) (net 5))
+  (segment (start -91.6 49.85) (end -90.425 51.025) (width 1) (layer F.Cu) (net 5))
+  (segment (start -98.425 48.675) (end -92.85 48.675) (width 1) (layer F.Cu) (net 5))
+  (segment (start -91.675 49.85) (end -91.6 49.85) (width 1) (layer F.Cu) (net 5))
+  (segment (start -92.85 48.675) (end -91.675 49.85) (width 1) (layer F.Cu) (net 5))
+  (segment (start -92.459 62.621) (end -92.19 62.89) (width 1) (layer F.Cu) (net 5))
+  (segment (start -92.459 57.984) (end -92.459 62.621) (width 1) (layer F.Cu) (net 5))
+  (segment (start -92.45 57.975) (end -92.459 57.984) (width 1) (layer F.Cu) (net 5))
+  (segment (start -92.45 57.7) (end -92.45 57.975) (width 1) (layer F.Cu) (net 5))
   (segment (start -112.12 33.095) (end -112.158 33.133) (width 1) (layer F.Cu) (net 6))
   (segment (start -112.919999 32.295001) (end -112.12 33.095) (width 1) (layer B.Cu) (net 6))
@@
   (segment (start -102.375 63.5) (end -98.6 63.5) (width 1) (layer B.Cu) (net 7))
   (segment (start -98.6 63.5) (end -95.17 60.07) (width 1) (layer B.Cu) (net 7))
-  (segment (start -94.583 56.3) (end -92.569 54.286) (width 1) (layer F.Cu) (net 7))
   (segment (start -94.795 56.3) (end -94.583 56.3) (width 1) (layer F.Cu) (net 7))
   (segment (start -95.17 56.675) (end -94.795 56.3) (width 1) (layer B.Cu) (net 7))
@@
   (segment (start -120.2 62.625) (end -120.172 62.597) (width 1) (layer B.Cu) (net 7))
   (segment (start -120.2 63.325) (end -120.2 62.625) (width 1) (layer B.Cu) (net 7))
+  (segment (start -92.569 54.991) (end -92.45 55.11) (width 1) (layer B.Cu) (net 7))
+  (segment (start -92.569 54.286) (end -92.569 54.991) (width 1) (layer B.Cu) (net 7))
+  (segment (start -93.605 55.11) (end -94.795 56.3) (width 1) (layer B.Cu) (net 7))
+  (segment (start -92.45 55.11) (end -93.605 55.11) (width 1) (layer B.Cu) (net 7))
   (segment (start -119.770001 65.595001) (end -118.036001 63.861001) (width 1) (layer B.Cu) (net 8))
   (segment (start -118.036001 63.861001) (end -117.961001 63.861001) (width 1) (layer B.Cu) (net 8))

Commit message: update
Parts:
- moved U3 0.20 mm to (-99.9, 56.5)
Routing:
- net VIN: track 81.0 -> 82.1 mm
- net D4: track 31.1 -> 32.1 mm
- net D5: track 40.7 -> 39.9 mm

Commit message: update
Parts:
- moved G*** 0.11 mm to (-114.2, 7.22)
Changed lines of the file:
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@@
   )
   (module footprints:moth4 (layer F.Cu)
-    (at -114.13 7.32 30)
+    (at -114.18 7.22 30)
     (fp_text reference G*** (at 0 0 30) (layer F.SilkS) hide
       (effects (font (size 1.524 1.524) (thickness 0.3)))
@@
     (descr "Resistor, Axial_DIN0204 series, Axial, Horizontal, pin pitch=7.62mm, 0.167W, length*diameter=3.6*1.6mm^2, http://cdn-reichelt.de/documents/datenblatt/B400/1_4W%23YAG.pdf")
     (tags "Resistor Axial_DIN0204 series Axial Horizontal pin pitch 7.62mm 0.167W length 3.6mm diameter 1.6mm")
-    (fp_text reference R2 (at 3.775 1.85 90) (layer F.SilkS)
+    (fp_text reference R2 (at 3.76 1.87 90) (layer F.SilkS)
       (effects (font (size 1 1) (thickness 0.15)))
     )
@@
     (descr "CP, Radial series, Radial, pin pitch=2.50mm, , diameter=5mm, Electrolytic Capacitor")
     (tags "CP Radial series Radial pin pitch 2.50mm  diameter 5mm Electrolytic Capacitor")
-    (fp_text reference C5 (at -1.565 2.365 180) (layer F.SilkS)
+    (fp_text reference C5 (at -1.385 2.265 220) (layer F.SilkS)
       (effects (font (size 1 1) (thickness 0.15)))
     )
@@
     (effects (font (size 0.85 0.85) (thickness 0.15)))
   )
-  (gr_text http://pvos.org/ (at -124.08 7.85) (layer F.SilkS)
+  (gr_text http://pvos.org/ (at -124.09 7.61) (layer F.SilkS)
     (effects (font (size 1.1 1.1) (thickness 0.15)))
   )
@@
     (effects (font (size 0.8 0.8) (thickness 0.15)))
   )
-  (gr_text v4 (at -116.03 12.55) (layer F.SilkS)
+  (gr_text v4 (at -114.04 11.22) (layer F.SilkS)
     (effects (font (size 1 1) (thickness 0.15)))
   )

Commit message: update
Parts:
- moved G*** 2.36 mm to (-114.6, 9.54), turned to 300 degrees
Other:
- board text added: "A4"
- board text added: "A5"
Changed lines of the file:
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@@
   (general
     (thickness 1.6)
-    (drawings 88)
+    (drawings 90)
     (tracks 644)
     (zones 0)
@@
   )
   (module footprints:moth4 (layer F.Cu)
-    (at -114.18 7.22 30)
-    (fp_text reference G*** (at 0 0 30) (layer F.SilkS) hide
+    (at -114.62 9.54 300)
+    (fp_text reference G*** (at 0 0 120) (layer F.SilkS) hide
       (effects (font (size 1.524 1.524) (thickness 0.3)))
     )
-    (fp_text value LOGO (at 0.75 0 30) (layer F.SilkS) hide
+    (fp_text value LOGO (at 0.75 0 120) (layer F.SilkS) hide
       (effects (font (size 1.524 1.524) (thickness 0.3)))
     )
@@
     )
   )
+  (gr_text A5 (at -128.73 45.35 270) (layer F.SilkS)
+    (effects (font (size 0.8 0.8) (thickness 0.15)))
+  )
+  (gr_text A4 (at -128.69 40.35 270) (layer F.SilkS)
+    (effects (font (size 0.8 0.8) (thickness 0.15)))
+  )
   (gr_line (start -108.23 50.31) (end -107.83 49.67) (layer F.SilkS) (width 0.12))
   (gr_line (start -108.23 50.27) (end -108.7 49.63) (layer F.SilkS) (width 0.12))
@@
     (effects (font (size 1.1 1.1) (thickness 0.15)))
   )
-  (gr_text GND (at -92.96 76.46) (layer F.SilkS)
+  (gr_text GND (at -92.91 76.42) (layer F.SilkS)
     (effects (font (size 1.1 1.1) (thickness 0.15)))
   )
-  (gr_text VIN (at -96.64 76.43) (layer F.SilkS)
+  (gr_text VIN (at -96.53 76.42) (layer F.SilkS)
     (effects (font (size 1.1 1.1) (thickness 0.15)))
   )
@@
     (effects (font (size 0.85 0.85) (thickness 0.15)))
   )
-  (gr_text http://pvos.org/ (at -124.09 7.61) (layer F.SilkS)
+  (gr_text http://pvos.org/ (at -123.07 7.72) (layer F.SilkS)
     (effects (font (size 1.1 1.1) (thickness 0.15)))
   )
@@
     (effects (font (size 0.8 0.8) (thickness 0.15)))
   )
-  (gr_text v4 (at -114.04 11.22) (layer F.SilkS)
+  (gr_text v4 (at -115.52 11.63) (layer F.SilkS)
     (effects (font (size 1 1) (thickness 0.15)))
   )
-  (gr_text MOTHBOT (at -122.97 10.39) (layer F.SilkS)
-    (effects (font (size 2.5 2.5) (thickness 0.3)))
+  (gr_text MOTHBOT (at -123.73 10.34) (layer F.SilkS)
+    (effects (font (size 2.2 2.2) (thickness 0.3)))
   )
   (gr_text RST (at -121.5 13.4 180) (layer B.SilkS)
@@
     (effects (font (size 1.1 1.1) (thickness 0.15)))
   )
-  (gr_text GND (at -85.725 67.025 90) (layer F.SilkS)
+  (gr_text GND (at -85.76 67.76 90) (layer F.SilkS)
     (effects (font (size 1.1 1.1) (thickness 0.15)))
   )
-  (gr_text VIN (at -85.7 61.95 90) (layer F.SilkS)
+  (gr_text VIN (at -85.71 62.92 90) (layer F.SilkS)
     (effects (font (size 1.1 1.1) (thickness 0.15)))
   )

Commit message: update
Parts:
- moved G*** 0.21 mm to (-114.7, 9.33)
Routing:
- net A3: track 106.9 -> 102.0 mm
Other:
- board text added: "(U1 top / notch)"
- board text removed: "(U1 'top')"
Changed lines of the file:
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@@
     (thickness 1.6)
     (drawings 90)
-    (tracks 644)
+    (tracks 640)
     (zones 0)
     (modules 40)
@@
   )
   (module footprints:moth4 (layer F.Cu)
-    (at -114.62 9.54 300)
+    (at -114.65 9.33 300)
     (fp_text reference G*** (at 0 0 120) (layer F.SilkS) hide
       (effects (font (size 1.524 1.524) (thickness 0.3)))
@@
     (descr "Through hole straight socket strip, 1x04, 2.54mm pitch, single row (from Kicad 4.0.7), script generated")
     (tags "Through hole socket strip THT 1x04 2.54mm single row")
-    (fp_text reference J11 (at 0.205 -2.45 90) (layer F.SilkS)
+    (fp_text reference J11 (at 0.205 -2.45 270) (layer F.SilkS)
       (effects (font (size 1 1) (thickness 0.15)))
     )
@@
     (descr "Terminal Block Phoenix MKDS-1,5-6, 6 pins, pitch 5mm, size 30x9.8mm^2, drill diamater 1.3mm, pad diameter 2.6mm, see http://www.farnell.com/datasheets/100425.pdf, script-generated using https://github.com/pointhi/kicad-footprint-generator/scripts/TerminalBlock_Phoenix")
     (tags "THT Terminal Block Phoenix MKDS-1,5-6 pitch 5mm size 30x9.8mm^2 drill 1.3mm pad 2.6mm")
-    (fp_text reference J3 (at -3.51 -3.4 180) (layer F.SilkS)
+    (fp_text reference J3 (at -3.37 -3.54 180) (layer F.SilkS)
       (effects (font (size 1 1) (thickness 0.15)))
     )
@@
     (descr "C, Disc series, Radial, pin pitch=5.00mm, , diameter*width=4.3*1.9mm^2, Capacitor, http://www.vishay.com/docs/45233/krseries.pdf")
     (tags "C Disc series Radial pin pitch 5.00mm  diameter 4.3mm width 1.9mm Capacitor")
-    (fp_text reference C6 (at 6.75 -0.1 270) (layer F.SilkS)
+    (fp_text reference C6 (at 6.89 -0.125 270) (layer F.SilkS)
       (effects (font (size 1 1) (thickness 0.15)))
     )
@@
     (descr "Through hole straight socket strip, 1x03, 2.54mm pitch, single row (from Kicad 4.0.7), script generated")
     (tags "Through hole socket strip THT 1x03 2.54mm single row")
-    (fp_text reference J9 (at 1.003 9.289 270) (layer F.SilkS)
+    (fp_text reference J9 (at -4.427 9.224 270) (layer F.SilkS)
       (effects (font (size 1 1) (thickness 0.15)))
     )
@@
     (tags "SMA Straight Samtec Edge Mount")
     (attr smd)
-    (fp_text reference J4 (at 4.595 1.521) (layer F.SilkS)
+    (fp_text reference J4 (at 4.31 1.241 90) (layer F.SilkS)
       (effects (font (size 1 1) (thickness 0.15)))
     )
@@
     (descr "Terminal Block Phoenix PT-1,5-2-5.0-H, 2 pins, pitch 5mm, size 10x9mm^2, drill diamater 1.3mm, pad diameter 2.6mm, see http://www.mouser.com/ds/2/324/ItemDetail_1935161-922578.pdf, script-generated using https://github.com/pointhi/kicad-footprint-generator/scripts/TerminalBlock_Phoenix")
     (tags "THT Terminal Block Phoenix PT-1,5-2-5.0-H pitch 5mm size 10x9mm^2 drill 1.3mm pad 2.6mm")
-    (fp_text reference J1 (at 8.295 -1.345) (layer F.SilkS)
+    (fp_text reference J1 (at 8.23 -2.35) (layer F.SilkS)
       (effects (font (size 1 1) (thickness 0.15)))
     )
@@
   (gr_circle (center -128.58 1.27) (end -126.4 3.21) (layer F.SilkS) (width 0.12))
   (gr_circle (center -87.84 1.21) (end -85.5 3.03) (layer F.SilkS) (width 0.12))
-  (gr_text "(U1 'top')" (at -108.28 45.29 90) (layer F.SilkS)
+  (gr_text "(U1 top / notch)" (at -108.21 43.55 90) (layer F.SilkS)
     (effects (font (size 0.8 0.8) (thickness 0.15)))
   )
@@
     (effects (font (size 0.8 0.8) (thickness 0.15)))
   )
-  (gr_text v4 (at -115.52 11.63) (layer F.SilkS)
-    (effects (font (size 1 1) (thickness 0.15)))
+  (gr_text v4 (at -115.71 12.05) (layer F.SilkS)
+    (effects (font (size 1.2 1.2) (thickness 0.15)))
   )
   (gr_text MOTHBOT (at -123.73 10.34) (layer F.SilkS)
@@
     (effects (font (size 1.1 1.1) (thickness 0.15)))
   )
-  (gr_text GND (at -130.675 16 270) (layer F.SilkS)
+  (gr_text GND (at -130.56 15.98 270) (layer F.SilkS)
     (effects (font (size 1.1 1.1) (thickness 0.15)))
   )
@@
     (effects (font (size 0.85 0.85) (thickness 0.15)))
   )
-  (gr_text VIN (at -101.765 48.865) (layer F.SilkS)
+  (gr_text VIN (at -101.75 48.93) (layer F.SilkS)
     (effects (font (size 0.85 0.85) (thickness 0.15)))
   )
-  (gr_text RESET (at -130.19 65.98 270) (layer F.SilkS)
+  (gr_text RESET (at -129.84 65.78 270) (layer F.SilkS)
     (effects (font (size 1.3 1.3) (thickness 0.15)))
   )
@@
   (segment (start -98.6 63.5) (end -102.375 63.5) (width 1) (layer B.Cu) (net 7))
   (segment (start -94.81 59.71) (end -98.6 63.5) (width 1) (layer B.Cu) (net 7))
-  (segment (start -119.770001 65.595001) (end -118.036001 63.861001) (width 1) (layer B.Cu) (net 8))
-  (segment (start -118.036001 63.861001) (end -117.961001 63.861001) (width 1) (layer B.Cu) (net 8))
-  (segment (start -117.961001 63.861001) (end -116.875 62.775) (width 1) (layer B.Cu) (net 8))
-  (segment (start -119.770001 66.445001) (end -119.770001 65.595001) (width 1) (layer B.Cu) (net 8))
   (segment (start -112.12 45.795) (end -114.205 45.795) (width 1) (layer B.Cu) (net 8))
   (segment (start -114.205 45.795) (end -117.375 42.625) (width 1) (layer B.Cu) (net 8))

Commit message: update
Parts:
- moved R4 2.24 mm to (-97.6, 63.2)
- moved R5 1.88 mm to (-99.9, 69.8)
- moved J1 0.54 mm to (-91.7, 67.8)
Routing:
- net VIN: track 82.1 -> 73.0 mm
- net VCC: track 212.9 -> 216.2 mm
- net GND: track 341.3 -> 342.6 mm
- net RX0: track 30.7 -> 31.5 mm
- net A3: track 102.0 -> 101.5 mm
Other:
- board text added: "1"
- board text added: "14"
- board text added: "28"
